File: KiCAD_files/Driver.sch (KiCad schematic (older format))
At the start: 37 parts, among them J1 Driver_stage_outline_outputs, J2 Driver_stage_outline_inputs, U12 SFH617A-2X009T, U3 UCC21520DW, U4 UCC21520DW

Commit message: Improved power board traces - Took a power electronic routing guideline into consideration.
Parts:
- removed D_Boot1, D_Boot2: D_Schottky_AKA, Diode_SMD:D_SMB, symbol Device:D_Schottky_AKA
- added D_boot1, D_boot2: D_Schottky, Diode_SMD:D_SMB, symbol Device:D_Schottky
Connections:
- net labels added: +5VD
- net labels removed: +5C
- wire segments 133 -> 131
Changed lines of the file:
@@
 Wire Wire Line
 	2000 6200 2000 6350
-$Comp
-L power:+5C #PWR0110
-U 1 1 5EA37204
-P 2550 5600
-AR Path="/5EA37204" Ref="#PWR0110"  Part="1"
-AR Path="/5E9944F3/5EA37204" Ref="#PWR0116"  Part="1"
-F 0 "#PWR0110" H 2550 5450 50  0001 C CNN
-F 1 "+5C" H 2565 5773 50  0000 C CNN
-F 2 "" H 2550 5600 50  0001 C CNN
-F 3 "" H 2550 5600 50  0001 C CNN
-	1    2550 5600
-	1    0    0    -1
-$EndComp
 Wire Wire Line
 	2550 5600 2850 5600
@@
 	2700 6700 2550 6700
 Connection ~ 2400 6700
-$Comp
-L power:+5C #PWR0111
-U 1 1 5EA37224
-P 2550 7100
-AR Path="/5EA37224" Ref="#PWR0111"  Part="1"
-AR Path="/5E9944F3/5EA37224" Ref="#PWR0117"  Part="1"
-F 0 "#PWR0111" H 2550 6950 50  0001 C CNN
-F 1 "+5C" H 2565 7273 50  0000 C CNN
-F 2 "" H 2550 7100 50  0001 C CNN
-F 3 "" H 2550 7100 50  0001 C CNN
-	1    2550 7100
-	1    0    0    1
-$EndComp
 Wire Wire Line
 	2400 6900 2550 6900
@@
 Wire Wire Line
 	2550 6400 2550 6700
-$Comp
-L Device:D_Schottky_AKA D_Boot1
-U 1 1 5EA37288
-P 4250 4950
-AR Path="/5EA37288" Ref="D_Boot1"  Part="1"
-AR Path="/5E9944F3/5EA37288" Ref="D_Boot1"  Part="1"
-F 0 "D_Boot1" V 4321 5091 50  0000 L CNN
-F 1 "D_Schottky_AKA" V 4230 5091 50  0000 L CNN
-F 2 "Diode_SMD:D_SMB" H 4250 4950 50  0001 C CNN
-F 3 "~" H 4250 4950 50  0001 C CNN
-	1    4250 4950
-	0    1    -1   0
-$EndComp
-Wire Wire Line
-	4350 4750 4250 4750
-Connection ~ 4250 4750
 Wire Wire Line
 	1750 5900 2000 5900
@@
 Wire Wire Line
 	7450 6200 7450 6350
-$Comp
-L power:+5C #PWR0141
-U 1 1 5F2CDD56
-P 8000 5600
-AR Path="/5F2CDD56" Ref="#PWR0141"  Part="1"
-AR Path="/5E9944F3/5F2CDD56" Ref="#PWR0154"  Part="1"
-F 0 "#PWR0141" H 8000 5450 50  0001 C CNN
-F 1 "+5C" H 8015 5773 50  0000 C CNN
-F 2 "" H 8000 5600 50  0001 C CNN
-F 3 "" H 8000 5600 50  0001 C CNN
-	1    8000 5600
-	1    0    0    -1
-$EndComp
 Wire Wire Line
 	8000 5600 8300 5600
@@
 	8150 6700 8000 6700
 Connection ~ 7850 6700
-$Comp
-L power:+5C #PWR0142
-U 1 1 5F2CDD73
-P 8000 7100
-AR Path="/5F2CDD73" Ref="#PWR0142"  Part="1"
-AR Path="/5E9944F3/5F2CDD73" Ref="#PWR0158"  Part="1"
-F 0 "#PWR0142" H 8000 6950 50  0001 C CNN
-F 1 "+5C" H 8015 7273 50  0000 C CNN
-F 2 "" H 8000 7100 50  0001 C CNN
-F 3 "" H 8000 7100 50  0001 C CNN
-	1    8000 7100
-	1    0    0    1
-$EndComp
 Wire Wire Line
 	7850 6900 8000 6900
@@
 Wire Wire Line
 	8000 6400 8000 6700
-$Comp
-L Device:D_Schottky_AKA D_Boot2
-U 1 1 5F2CDDA0
-P 9700 4950
-AR Path="/5F2CDDA0" Ref="D_Boot2"  Part="1"
-AR Path="/5E9944F3/5F2CDDA0" Ref="D_Boot2"  Part="1"
-F 0 "D_Boot2" V 9771 5091 50  0000 L CNN
-F 1 "D_Schottky_AKA" V 9680 5091 50  0000 L CNN
-F 2 "Diode_SMD:D_SMB" H 9700 4950 50  0001 C CNN
-F 3 "~" H 9700 4950 50  0001 C CNN
-	1    9700 4950
-	0    1    -1   0
-$EndComp
-Wire Wire Line
-	9800 4750 9700 4750
-Connection ~ 9700 4750
 Wire Wire Line
 	7200 5900 7450 5900
@@
 Connection ~ 10500 5800
 Wire Wire Line
-	9700 5100 9700 5150
-Wire Wire Line
 	10500 5250 10500 5150
 Wire Wire Line
@@
 Wire Wire Line
 	9950 5150 9700 5150
-Wire Wire Line
-	4250 5100 4250 5200
 Connection ~ 4250 5200
 Wire Wire Line
@@
 Text Label 1200 6000 0    50   ~ 0
 PWM_L1_D
-$Comp
-L power:+5C #PWR0117
-U 1 1 5F48BDEB
-P 5650 1550
-AR Path="/5F48BDEB" Ref="#PWR0117"  Part="1"
-AR Path="/5E9944F3/5F48BDEB" Ref="#PWR?"  Part="1"
-F 0 "#PWR0117" H 5650 1400 50  0001 C CNN
-F 1 "+5C" H 5665 1723 50  0000 C CNN
-F 2 "" H 5650 1550 50  0001 C CNN
-F 3 "" H 5650 1550 50  0001 C CNN
-	1    5650 1550
-	0    -1   -1   0
-$EndComp
-$Comp
-L power:+5C #PWR0118
-U 1 1 5F491752
-P 5650 2150
-AR Path="/5F491752" Ref="#PWR0118"  Part="1"
-AR Path="/5E9944F3/5F491752" Ref="#PWR?"  Part="1"
-F 0 "#PWR0118" H 5650 2000 50  0001 C CNN
-F 1 "+5C" H 5665 2323 50  0000 C CNN
-F 2 "" H 5650 2150 50  0001 C CNN
-F 3 "" H 5650 2150 50  0001 C CNN
-	1    5650 2150
-	0    -1   -1   0
-$EndComp
 Wire Wire Line
 	5650 1550 5800 1550
@@
 Wire Wire Line
 	3800 1750 3200 1750
+$Comp
+L power:+5VD #PWR0110
+U 1 1 5F4DF8B9
+P 5650 1550
+F 0 "#PWR0110" H 5650 1400 50  0001 C CNN
+F 1 "+5VD" V 5665 1678 50  0000 L CNN
+F 2 "" H 5650 1550 50  0001 C CNN
+F 3 "" H 5650 1550 50  0001 C CNN
+	1    5650 1550
+	0    -1   -1   0
+$EndComp
+$Comp
+L power:+5VD #PWR0111
+U 1 1 5F4E05F4
+P 5650 2150
+F 0 "#PWR0111" H 5650 2000 50  0001 C CNN
+F 1 "+5VD" V 5665 2278 50  0000 L CNN
+F 2 "" H 5650 2150 50  0001 C CNN
+F 3 "" H 5650 2150 50  0001 C CNN
+	1    5650 2150
+	0    -1   -1   0
+$EndComp
+$Comp
+L power:+5VD #PWR0117
+U 1 1 5F4FEB42
+P 2550 5600
+F 0 "#PWR0117" H 2550 5450 50  0001 C CNN
+F 1 "+5VD" V 2565 5728 50  0000 L CNN
+F 2 "" H 2550 5600 50  0001 C CNN
+F 3 "" H 2550 5600 50  0001 C CNN
+	1    2550 5600
+	0    -1   -1   0
+$EndComp
+$Comp
+L power:+5VD #PWR0118
+U 1 1 5F518358
+P 8000 5600
+F 0 "#PWR0118" H 8000 5450 50  0001 C CNN
+F 1 "+5VD" V 8015 5728 50  0000 L CNN
+F 2 "" H 8000 5600 50  0001 C CNN
+F 3 "" H 8000 5600 50  0001 C CNN
+	1    8000 5600
+	0    -1   -1   0
+$EndComp
+$Comp
+L power:+5VD #PWR0120
+U 1 1 5F5294F8
+P 8000 7100
+F 0 "#PWR0120" H 8000 6950 50  0001 C CNN
+F 1 "+5VD" V 8015 7228 50  0000 L CNN
+F 2 "" H 8000 7100 50  0001 C CNN
+F 3 "" H 8000 7100 50  0001 C CNN
+	1    8000 7100
+	0    -1   -1   0
+$EndComp
+$Comp
+L power:+5VD #PWR0121
+U 1 1 5F535163
+P 2550 7100
+F 0 "#PWR0121" H 2550 6950 50  0001 C CNN
+F 1 "+5VD" V 2565 7228 50  0000 L CNN
+F 2 "" H 2550 7100 50  0001 C CNN
+F 3 "" H 2550 7100 50  0001 C CNN
+	1    2550 7100
+	0    -1   -1   0
+$EndComp
+$Comp
+L Device:D_Schottky D_boot1
+U 1 1 5F53F341
+P 4250 4900
+F 0 "D_boot1" V 4296 4820 50  0000 R CNN
+F 1 "D_Schottky" V 4205 4820 50  0000 R CNN
+F 2 "Diode_SMD:D_SMB" H 4250 4900 50  0001 C CNN
+F 3 "~" H 4250 4900 50  0001 C CNN
+	1    4250 4900
+	0    -1   -1   0
+$EndComp
+Wire Wire Line
+	4250 5050 4250 5200
+$Comp
+L Device:D_Schottky D_boot2
+U 1 1 5F566B39
+P 9700 4900
+F 0 "D_boot2" V 9746 4820 50  0000 R CNN
+F 1 "D_Schottky" V 9655 4820 50  0000 R CNN
+F 2 "Diode_SMD:D_SMB" H 9700 4900 50  0001 C CNN
+F 3 "~" H 9700 4900 50  0001 C CNN
+	1    9700 4900
+	0    -1   -1   0
+$EndComp
+Wire Wire Line
+	9700 5050 9700 5150
 $EndSCHEMATC

Commit message: Improved driver schematic - added missing infos
Parts:
- U3, U4: value UCC21520DW -> UCC21222DR
Other:
- moved on the sheet: C_VDDB2, C_VDDB4
Changed lines of the file:
@@
 AR Path="/5E9944F3/5EA37157" Ref="U6"  Part="1"
 F 0 "U3" H 3350 6665 50  0000 C CNN
-F 1 "UCC21520DW" H 3350 6574 50  0000 C CNN
+F 1 "UCC21222DR" H 3350 6574 50  0000 C CNN
 F 2 "Package_SO:SOIC-16_3.9x9.9mm_P1.27mm" H 3350 5450 50  0001 C CNN
-F 3 "http://www.ti.com/lit/ds/symlink/ucc21520.pdf" H 3350 5950 50  0001 C CNN
+F 3 "http://www.ti.com/lit/ds/symlink/ucc21222.pdf" H 3350 5950 50  0001 C CNN
 	1    3350 6000
 	1    0    0    -1
@@
 AR Path="/5EA371B8" Ref="R1"  Part="1"
 AR Path="/5E9944F3/5EA371B8" Ref="R1"  Part="1"
-F 0 "R1" V 1846 5900 50  0000 C CNN
+F 0 "R1" V 1450 6000 50  0000 C CNN
 F 1 "R_Small" V 1755 5900 50  0000 C CNN
 F 2 "Resistor_SMD:R_0805_2012Metric" H 1650 5900 50  0001 C CNN
@@
 AR Path="/5EA371BF" Ref="R2"  Part="1"
 AR Path="/5E9944F3/5EA371BF" Ref="R2"  Part="1"
-F 0 "R2" H 1709 6046 50  0000 L CNN
-F 1 "R_Small" H 1709 5955 50  0000 L CNN
+F 0 "R2" V 1950 6050 50  0000 L CNN
+F 1 "R_Small" V 1450 5850 50  0000 L CNN
 F 2 "Resistor_SMD:R_0805_2012Metric" H 1650 6000 50  0001 C CNN
 F 3 "~" H 1650 6000 50  0001 C CNN
@@
 L power:GNDD #PWR0107
 U 1 1 5EA371EC
-P 2150 6800
+P 1900 6800
 AR Path="/5EA371EC" Ref="#PWR0107"  Part="1"
 AR Path="/5E9944F3/5EA371EC" Ref="#PWR0113"  Part="1"
-F 0 "#PWR0107" H 2150 6550 50  0001 C CNN
-F 1 "GNDD" H 2154 6645 50  0000 C CNN
-F 2 "" H 2150 6800 50  0001 C CNN
-F 3 "" H 2150 6800 50  0001 C CNN
-	1    2150 6800
+F 0 "#PWR0107" H 1900 6550 50  0001 C CNN
+F 1 "GNDD" H 1904 6645 50  0000 C CNN
+F 2 "" H 1900 6800 50  0001 C CNN
+F 3 "" H 1900 6800 50  0001 C CNN
+	1    1900 6800
 	1    0    0    -1
 $EndComp
@@
 AR Path="/5EA3720B" Ref="C3"  Part="1"
 AR Path="/5E9944F3/5EA3720B" Ref="C11"  Part="1"
-F 0 "C3" H 2492 6846 50  0000 L CNN
-F 1 "C_Small" H 2492 6755 50  0000 L CNN
+F 0 "C3" H 2050 6800 50  0000 L CNN
+F 1 "C_Small" H 2050 6700 50  0000 L CNN
 F 2 "Capacitor_SMD:C_0805_2012Metric" H 2400 6800 50  0001 C CNN
 F 3 "~" H 2400 6800 50  0001 C CNN
@@
 AR Path="/5EA37212" Ref="C4"  Part="1"
 AR Path="/5E9944F3/5EA37212" Ref="C12"  Part="1"
-F 0 "C4" H 2642 6846 50  0000 L CNN
-F 1 "C_Small" H 2642 6755 50  0000 L CNN
+F 0 "C4" H 2650 6650 50  0000 L CNN
+F 1 "C_Small" H 2650 6550 50  0000 L CNN
 F 2 "Capacitor_SMD:C_0805_2012Metric" H 2550 6800 50  0001 C CNN
 F 3 "~" H 2550 6800 50  0001 C CNN
@@
 AR Path="/5EA37219" Ref="C6"  Part="1"
 AR Path="/5E9944F3/5EA37219" Ref="C14"  Part="1"
-F 0 "C6" H 2792 6846 50  0000 L CNN
-F 1 "C_Small" H 2792 6755 50  0000 L CNN
+F 0 "C6" H 2950 6850 50  0000 L CNN
+F 1 "C_Small" H 2950 6750 50  0000 L CNN
 F 2 "Capacitor_SMD:C_0805_2012Metric" H 2700 6800 50  0001 C CNN
 F 3 "~" H 2700 6800 50  0001 C CNN
@@
 	2400 6100 2400 6700
 Wire Wire Line
-	2400 6700 2150 6700
-Wire Wire Line
-	2150 6700 2150 6800
+	2400 6700 1900 6700
+Wire Wire Line
+	1900 6700 1900 6800
 Wire Wire Line
 	2700 6300 2850 6300
@@
 L Device:C C_VDDB2
 U 1 1 5EA06D1F
-P 4150 7400
+P 4150 7600
 AR Path="/5EA06D1F" Ref="C_VDDB2"  Part="1"
 AR Path="/5E9944F3/5EA06D1F" Ref="C_VDDB2"  Part="1"
-F 0 "C_VDDB2" V 4402 7400 50  0000 C CNN
-F 1 "100nF" V 4311 7400 50  0000 C CNN
-F 2 "Capacitor_SMD:C_1210_3225Metric" H 4188 7250 50  0001 C CNN
-F 3 "~" H 4150 7400 50  0001 C CNN
-	1    4150 7400
-	0    -1   -1   0
-$EndComp
-Wire Wire Line
-	4000 7400 4000 7100
+F 0 "C_VDDB2" V 4402 7600 50  0000 C CNN
+F 1 "100nF" V 4311 7600 50  0000 C CNN
+F 2 "Capacitor_SMD:C_1210_3225Metric" H 4188 7450 50  0001 C CNN
+F 3 "~" H 4150 7600 50  0001 C CNN
+	1    4150 7600
+	0    -1   -1   0
+$EndComp
+Wire Wire Line
+	4000 7600 4000 7100
 Connection ~ 4000 7100
 Wire Wire Line
-	4300 7400 4300 7100
+	4300 7600 4300 7100
 Connection ~ 4300 7100
 Text Label 4350 9400 0    50   ~ 0
@@
 AR Path="/5E9944F3/5F2CDCCA" Ref="U14"  Part="1"
 F 0 "U4" H 8800 6665 50  0000 C CNN
-F 1 "UCC21520DW" H 8800 6574 50  0000 C CNN
+F 1 "UCC21222DR" H 8800 6574 50  0000 C CNN
 F 2 "Package_SO:SOIC-16_3.9x9.9mm_P1.27mm" H 8800 5450 50  0001 C CNN
-F 3 "http://www.ti.com/lit/ds/symlink/ucc21520.pdf" H 8800 5950 50  0001 C CNN
+F 3 "http://www.ti.com/lit/ds/symlink/ucc21222.pdf" H 8800 5950 50  0001 C CNN
 	1    8800 6000
-	1    0    0    -1
-$EndComp
-$Comp
-L power:GNDREF #PWR?
-U 1 1 5F2CDCD0
-P 10550 6550
-AR Path="/5E91AAF4/5F2CDCD0" Ref="#PWR?"  Part="1"
-AR Path="/5E86B783/5F2CDCD0" Ref="#PWR?"  Part="1"
-AR Path="/5F2CDCD0" Ref="#PWR0132"  Part="1"
-AR Path="/5E9944F3/5F2CDCD0" Ref="#PWR0138"  Part="1"
-F 0 "#PWR0132" H 10550 6300 50  0001 C CNN
-F 1 "GNDREF" H 10555 6377 50  0000 C CNN
-F 2 "" H 10550 6550 50  0001 C CNN
-F 3 "" H 10550 6550 50  0001 C CNN
-	1    10550 6550
 	1    0    0    -1
 $EndComp
@@
 AR Path="/5F2CDD2D" Ref="R7"  Part="1"
 AR Path="/5E9944F3/5F2CDD2D" Ref="R35"  Part="1"
-F 0 "R7" H 7159 6046 50  0000 L CNN
-F 1 "R_Small" H 7159 5955 50  0000 L CNN
+F 0 "R7" V 6850 5950 50  0000 L CNN
+F 1 "R_Small" V 6950 5950 50  0000 L CNN
 F 2 "Resistor_SMD:R_0805_2012Metric" H 7100 6000 50  0001 C CNN
 F 3 "~" H 7100 6000 50  0001 C CNN
@@
 L power:GNDD #PWR0138
 U 1 1 5F2CDD43
-P 7600 6800
+P 7150 6800
 AR Path="/5F2CDD43" Ref="#PWR0138"  Part="1"
 AR Path="/5E9944F3/5F2CDD43" Ref="#PWR0146"  Part="1"
-F 0 "#PWR0138" H 7600 6550 50  0001 C CNN
-F 1 "GNDD" H 7604 6645 50  0000 C CNN
-F 2 "" H 7600 6800 50  0001 C CNN
-F 3 "" H 7600 6800 50  0001 C CNN
-	1    7600 6800
+F 0 "#PWR0138" H 7150 6550 50  0001 C CNN
+F 1 "GNDD" H 7154 6645 50  0000 C CNN
+F 2 "" H 7150 6800 50  0001 C CNN
+F 3 "" H 7150 6800 50  0001 C CNN
+	1    7150 6800
 	1    0    0    -1
 $EndComp
@@
 AR Path="/5F2CDD5D" Ref="C9"  Part="1"
 AR Path="/5E9944F3/5F2CDD5D" Ref="C42"  Part="1"
-F 0 "C9" H 7942 6846 50  0000 L CNN
-F 1 "C_Small" H 7942 6755 50  0000 L CNN
+F 0 "C9" H 7450 6850 50  0000 L CNN
+F 1 "C_Small" H 7450 6750 50  0000 L CNN
 F 2 "Capacitor_SMD:C_0805_2012Metric" H 7850 6800 50  0001 C CNN
 F 3 "~" H 7850 6800 50  0001 C CNN
@@
 AR Path="/5F2CDD63" Ref="C10"  Part="1"
 AR Path="/5E9944F3/5F2CDD63" Ref="C43"  Part="1"
-F 0 "C10" H 8092 6846 50  0000 L CNN
-F 1 "C_Small" H 8092 6755 50  0000 L CNN
+F 0 "C10" H 8050 6650 50  0000 L CNN
+F 1 "C_Small" H 8050 6550 50  0000 L CNN
 F 2 "Capacitor_SMD:C_0805_2012Metric" H 8000 6800 50  0001 C CNN
 F 3 "~" H 8000 6800 50  0001 C CNN
@@
 AR Path="/5F2CDD69" Ref="C12"  Part="1"
 AR Path="/5E9944F3/5F2CDD69" Ref="C45"  Part="1"
-F 0 "C12" H 8242 6846 50  0000 L CNN
-F 1 "C_Small" H 8242 6755 50  0000 L CNN
+F 0 "C12" H 8300 6850 50  0000 L CNN
+F 1 "C_Small" H 8300 6750 50  0000 L CNN
 F 2 "Capacitor_SMD:C_0805_2012Metric" H 8150 6800 50  0001 C CNN
 F 3 "~" H 8150 6800 50  0001 C CNN
@@
 	7850 6100 7850 6700
 Wire Wire Line
-	7850 6700 7600 6700
-Wire Wire Line
-	7600 6700 7600 6800
+	7850 6700 7150 6700
+Wire Wire Line
+	7150 6700 7150 6800
 Wire Wire Line
 	8150 6300 8300 6300
@@
 	8150 6600 8150 6700
 Wire Wire Line
-	6650 5900 7000 5900
-Wire Wire Line
-	6650 6000 7000 6000
+	6450 5900 7000 5900
+Wire Wire Line
+	6450 6000 7000 6000
 $Comp
 L Device:R_Small R8
@@
 L Device:C C_VDDB4
 U 1 1 5F2CDDAB
-P 9600 7400
+P 9600 7550
 AR Path="/5F2CDDAB" Ref="C_VDDB4"  Part="1"
 AR Path="/5E9944F3/5F2CDDAB" Ref="C_VDDB4"  Part="1"
-F 0 "C_VDDB4" V 9852 7400 50  0000 C CNN
-F 1 "100nF" V 9761 7400 50  0000 C CNN
-F 2 "Capacitor_SMD:C_1210_3225Metric" H 9638 7250 50  0001 C CNN
-F 3 "~" H 9600 7400 50  0001 C CNN
-	1    9600 7400
-	0    -1   -1   0
-$EndComp
-Wire Wire Line
-	9450 7400 9450 7100
+F 0 "C_VDDB4" V 9852 7550 50  0000 C CNN
+F 1 "100nF" V 9761 7550 50  0000 C CNN
+F 2 "Capacitor_SMD:C_1210_3225Metric" H 9638 7400 50  0001 C CNN
+F 3 "~" H 9600 7550 50  0001 C CNN
+	1    9600 7550
+	0    -1   -1   0
+$EndComp
+Wire Wire Line
+	9450 7550 9450 7100
 Connection ~ 9450 7100
 Wire Wire Line
-	9750 7400 9750 7100
+	9750 7550 9750 7100
 Connection ~ 9750 7100
 Text Label 5200 2050 0    50   ~ 0
@@
 	1    0    0    -1
 $EndComp
-Text Label 6650 5900 0    50   ~ 0
+Text Label 6450 5900 0    50   ~ 0
 PWM_H2_D
-Text Label 6650 6000 0    50   ~ 0
+Text Label 6450 6000 0    50   ~ 0
 PWM_L2_D
 Wire Wire Line
 	2000 5550 2000 5700
 Wire Wire Line
-	1200 5900 1550 5900
-Wire Wire Line
-	1200 6000 1550 6000
-Text Label 1200 5900 0    50   ~ 0
+	1000 5900 1550 5900
+Wire Wire Line
+	1000 6000 1550 6000
+Text Label 1000 5900 0    50   ~ 0
 PWM_H1_D
-Text Label 1200 6000 0    50   ~ 0
+Text Label 1000 6000 0    50   ~ 0
 PWM_L1_D
 Wire Wire Line
