File: KiCAD_files/Driver.sch (KiCad schematic (older format))
At the start: 37 parts, among them J1 Driver_stage_outline_outputs, J2 Driver_stage_outline_inputs, U12 SFH617A-2X009T, U3 UCC21222DR, U4 UCC21222DR

Commit message: Added values and datasheets to driver stage
Parts:
- C1, C10, C2, C4, C7, C8: value C_Small -> 33pF
- C12, C3, C6, C9: value C_Small -> 100nF
- CBoot2, CBoot4: value 1uF -> 100nF
- C_VDDB2, C_VDDB4: value 100nF -> 10uF
- D_boot1, D_boot2: value D_Schottky -> STTH4R02U
- R1, R2, R4, R6, R7: value R_Small -> 51
- R3, R8: value R_Small -> 20k
- R5: value R_Small -> 1k
- RBoot1, RBoot2: value R -> 2.2
Changed lines of the file:
@@
 AR Path="/5E9944F3/5EA37173" Ref="RBoot1"  Part="1"
 F 0 "RBoot1" H 4180 4504 50  0000 R CNN
-F 1 "R" H 4180 4595 50  0000 R CNN
+F 1 "2.2" H 4180 4595 50  0000 R CNN
 F 2 "Resistor_SMD:R_0805_2012Metric" V 4180 4550 50  0001 C CNN
 F 3 "~" H 4250 4550 50  0001 C CNN
@@
 AR Path="/5EA371B8" Ref="R1"  Part="1"
 AR Path="/5E9944F3/5EA371B8" Ref="R1"  Part="1"
-F 0 "R1" V 1450 6000 50  0000 C CNN
-F 1 "R_Small" V 1755 5900 50  0000 C CNN
+F 0 "R1" V 1350 6000 50  0000 C CNN
+F 1 "51" V 1755 5900 50  0000 C CNN
 F 2 "Resistor_SMD:R_0805_2012Metric" H 1650 5900 50  0001 C CNN
 F 3 "~" H 1650 5900 50  0001 C CNN
@@
 AR Path="/5E9944F3/5EA371BF" Ref="R2"  Part="1"
 F 0 "R2" V 1950 6050 50  0000 L CNN
-F 1 "R_Small" V 1450 5850 50  0000 L CNN
+F 1 "51" V 1550 5950 50  0000 L CNN
 F 2 "Resistor_SMD:R_0805_2012Metric" H 1650 6000 50  0001 C CNN
 F 3 "~" H 1650 6000 50  0001 C CNN
@@
 AR Path="/5E9944F3/5EA371DA" Ref="C6"  Part="1"
 F 0 "C1" H 2092 5846 50  0000 L CNN
-F 1 "C_Small" H 2092 5755 50  0000 L CNN
+F 1 "33pF" H 2092 5755 50  0000 L CNN
 F 2 "Capacitor_SMD:C_0805_2012Metric" H 2000 5800 50  0001 C CNN
 F 3 "~" H 2000 5800 50  0001 C CNN
@@
 AR Path="/5E9944F3/5EA371E3" Ref="C7"  Part="1"
 F 0 "C2" H 2092 6146 50  0000 L CNN
-F 1 "C_Small" H 2092 6055 50  0000 L CNN
+F 1 "33pF" H 2092 6055 50  0000 L CNN
 F 2 "Capacitor_SMD:C_0805_2012Metric" H 2000 6100 50  0001 C CNN
 F 3 "~" H 2000 6100 50  0001 C CNN
@@
 AR Path="/5E9944F3/5EA3720B" Ref="C11"  Part="1"
 F 0 "C3" H 2050 6800 50  0000 L CNN
-F 1 "C_Small" H 2050 6700 50  0000 L CNN
+F 1 "100nF" H 2050 6700 50  0000 L CNN
 F 2 "Capacitor_SMD:C_0805_2012Metric" H 2400 6800 50  0001 C CNN
 F 3 "~" H 2400 6800 50  0001 C CNN
@@
 AR Path="/5E9944F3/5EA37212" Ref="C12"  Part="1"
 F 0 "C4" H 2650 6650 50  0000 L CNN
-F 1 "C_Small" H 2650 6550 50  0000 L CNN
+F 1 "33pF" H 2650 6550 50  0000 L CNN
 F 2 "Capacitor_SMD:C_0805_2012Metric" H 2550 6800 50  0001 C CNN
 F 3 "~" H 2550 6800 50  0001 C CNN
@@
 AR Path="/5EA37219" Ref="C6"  Part="1"
 AR Path="/5E9944F3/5EA37219" Ref="C14"  Part="1"
-F 0 "C6" H 2950 6850 50  0000 L CNN
-F 1 "C_Small" H 2950 6750 50  0000 L CNN
+F 0 "C6" H 2900 6800 50  0000 L CNN
+F 1 "100nF" H 2900 6700 50  0000 L CNN
 F 2 "Capacitor_SMD:C_0805_2012Metric" H 2700 6800 50  0001 C CNN
 F 3 "~" H 2700 6800 50  0001 C CNN
@@
 AR Path="/5EA37236" Ref="C5"  Part="1"
 AR Path="/5E9944F3/5EA37236" Ref="C13"  Part="1"
-F 0 "C5" H 2792 6546 50  0000 L CNN
-F 1 "10nF" H 2792 6455 50  0000 L CNN
+F 0 "C5" H 2900 6450 50  0000 L CNN
+F 1 "10nF" H 2900 6350 50  0000 L CNN
 F 2 "Capacitor_SMD:C_0805_2012Metric" H 2700 6500 50  0001 C CNN
 F 3 "~" H 2700 6500 50  0001 C CNN
@@
 Wire Wire Line
 	2700 6600 2700 6700
-$Comp
-L Device:R_Small R3
-U 1 1 5EA3727C
-P 2550 6300
-AR Path="/5EA3727C" Ref="R3"  Part="1"
-AR Path="/5E9944F3/5EA3727C" Ref="R5"  Part="1"
-F 0 "R3" H 2609 6346 50  0000 L CNN
-F 1 "R_Small" H 2609 6255 50  0000 L CNN
-F 2 "Resistor_SMD:R_0805_2012Metric" H 2550 6300 50  0001 C CNN
-F 3 "~" H 2550 6300 50  0001 C CNN
-	1    2550 6300
-	-1   0    0    1
-$EndComp
 Wire Wire Line
 	2700 6150 2550 6150
@@
 AR Path="/5E9944F3/5EA06D1F" Ref="C_VDDB2"  Part="1"
 F 0 "C_VDDB2" V 4402 7600 50  0000 C CNN
-F 1 "100nF" V 4311 7600 50  0000 C CNN
+F 1 "10uF" V 4311 7600 50  0000 C CNN
 F 2 "Capacitor_SMD:C_1210_3225Metric" H 4188 7450 50  0001 C CNN
 F 3 "~" H 4150 7600 50  0001 C CNN
@@
 AR Path="/5E9944F3/5EBFD9F2" Ref="R32"  Part="1"
 F 0 "R5" H 4009 9646 50  0000 L CNN
-F 1 "R_Small" H 4009 9555 50  0000 L CNN
+F 1 "1k" H 4009 9555 50  0000 L CNN
 F 2 "Resistor_SMD:R_0805_2012Metric" H 3950 9600 50  0001 C CNN
 F 3 "~" H 3950 9600 50  0001 C CNN
@@
 AR Path="/5E9944F3/5EC17146" Ref="R4"  Part="1"
 F 0 "R4" H 3009 9646 50  0000 L CNN
-F 1 "R_Small" H 3009 9555 50  0000 L CNN
+F 1 "51" H 3009 9555 50  0000 L CNN
 F 2 "Resistor_SMD:R_0805_2012Metric" H 2950 9600 50  0001 C CNN
 F 3 "~" H 2950 9600 50  0001 C CNN
@@
 AR Path="/5E9944F3/5F2CDCE5" Ref="RBoot2"  Part="1"
 F 0 "RBoot2" H 9630 4504 50  0000 R CNN
-F 1 "R" H 9630 4595 50  0000 R CNN
+F 1 "2.2" H 9630 4595 50  0000 R CNN
 F 2 "Resistor_SMD:R_0805_2012Metric" V 9630 4550 50  0001 C CNN
 F 3 "~" H 9700 4550 50  0001 C CNN
@@
 AR Path="/5E9944F3/5F2CDD27" Ref="R33"  Part="1"
 F 0 "R6" V 7296 5900 50  0000 C CNN
-F 1 "R_Small" V 7205 5900 50  0000 C CNN
+F 1 "51" V 7205 5900 50  0000 C CNN
 F 2 "Resistor_SMD:R_0805_2012Metric" H 7100 5900 50  0001 C CNN
 F 3 "~" H 7100 5900 50  0001 C CNN
@@
 AR Path="/5E9944F3/5F2CDD2D" Ref="R35"  Part="1"
 F 0 "R7" V 6850 5950 50  0000 L CNN
-F 1 "R_Small" V 6950 5950 50  0000 L CNN
+F 1 "51" V 6950 5950 50  0000 L CNN
 F 2 "Resistor_SMD:R_0805_2012Metric" H 7100 6000 50  0001 C CNN
 F 3 "~" H 7100 6000 50  0001 C CNN
@@
 AR Path="/5E9944F3/5F2CDD34" Ref="C40"  Part="1"
 F 0 "C7" H 7542 5846 50  0000 L CNN
-F 1 "C_Small" H 7542 5755 50  0000 L CNN
+F 1 "33pF" H 7542 5755 50  0000 L CNN
 F 2 "Capacitor_SMD:C_0805_2012Metric" H 7450 5800 50  0001 C CNN
 F 3 "~" H 7450 5800 50  0001 C CNN
@@
 AR Path="/5E9944F3/5F2CDD3C" Ref="C41"  Part="1"
 F 0 "C8" H 7542 6146 50  0000 L CNN
-F 1 "C_Small" H 7542 6055 50  0000 L CNN
+F 1 "33pF" H 7542 6055 50  0000 L CNN
 F 2 "Capacitor_SMD:C_0805_2012Metric" H 7450 6100 50  0001 C CNN
 F 3 "~" H 7450 6100 50  0001 C CNN
@@
 AR Path="/5E9944F3/5F2CDD5D" Ref="C42"  Part="1"
 F 0 "C9" H 7450 6850 50  0000 L CNN
-F 1 "C_Small" H 7450 6750 50  0000 L CNN
+F 1 "100nF" H 7450 6750 50  0000 L CNN
 F 2 "Capacitor_SMD:C_0805_2012Metric" H 7850 6800 50  0001 C CNN
 F 3 "~" H 7850 6800 50  0001 C CNN
@@
 AR Path="/5E9944F3/5F2CDD63" Ref="C43"  Part="1"
 F 0 "C10" H 8050 6650 50  0000 L CNN
-F 1 "C_Small" H 8050 6550 50  0000 L CNN
+F 1 "33pF" H 8050 6550 50  0000 L CNN
 F 2 "Capacitor_SMD:C_0805_2012Metric" H 8000 6800 50  0001 C CNN
 F 3 "~" H 8000 6800 50  0001 C CNN
@@
 AR Path="/5F2CDD69" Ref="C12"  Part="1"
 AR Path="/5E9944F3/5F2CDD69" Ref="C45"  Part="1"
-F 0 "C12" H 8300 6850 50  0000 L CNN
-F 1 "C_Small" H 8300 6750 50  0000 L CNN
+F 0 "C12" H 8250 6850 50  0000 L CNN
+F 1 "100nF" H 8250 6750 50  0000 L CNN
 F 2 "Capacitor_SMD:C_0805_2012Metric" H 8150 6800 50  0001 C CNN
 F 3 "~" H 8150 6800 50  0001 C CNN
@@
 AR Path="/5F2CDD85" Ref="C11"  Part="1"
 AR Path="/5E9944F3/5F2CDD85" Ref="C44"  Part="1"
-F 0 "C11" H 8242 6546 50  0000 L CNN
-F 1 "10nF" H 8242 6455 50  0000 L CNN
+F 0 "C11" H 8350 6450 50  0000 L CNN
+F 1 "10nF" H 8350 6350 50  0000 L CNN
 F 2 "Capacitor_SMD:C_0805_2012Metric" H 8150 6500 50  0001 C CNN
 F 3 "~" H 8150 6500 50  0001 C CNN
@@
 AR Path="/5F2CDD95" Ref="R8"  Part="1"
 AR Path="/5E9944F3/5F2CDD95" Ref="R43"  Part="1"
-F 0 "R8" H 8059 6346 50  0000 L CNN
-F 1 "R_Small" H 8059 6255 50  0000 L CNN
+F 0 "R8" H 8200 6400 50  0000 L CNN
+F 1 "20k" H 8200 6300 50  0000 L CNN
 F 2 "Resistor_SMD:R_0805_2012Metric" H 8000 6300 50  0001 C CNN
 F 3 "~" H 8000 6300 50  0001 C CNN
@@
 AR Path="/5E9944F3/5F2CDDAB" Ref="C_VDDB4"  Part="1"
 F 0 "C_VDDB4" V 9852 7550 50  0000 C CNN
-F 1 "100nF" V 9761 7550 50  0000 C CNN
+F 1 "10uF" V 9761 7550 50  0000 C CNN
 F 2 "Capacitor_SMD:C_1210_3225Metric" H 9638 7400 50  0001 C CNN
 F 3 "~" H 9600 7550 50  0001 C CNN
@@
 AR Path="/5E9944F3/5F2CDDB5" Ref="CBoot4"  Part="1"
 F 0 "CBoot4" H 10615 5446 50  0000 L CNN
-F 1 "1uF" H 10615 5355 50  0000 L CNN
+F 1 "100nF" H 10615 5355 50  0000 L CNN
 F 2 "Capacitor_SMD:C_0805_2012Metric" H 10538 5250 50  0001 C CNN
 F 3 "~" H 10500 5400 50  0001 C CNN
@@
 AR Path="/5E9944F3/5EA191EA" Ref="CBoot2"  Part="1"
 F 0 "CBoot2" H 5265 5496 50  0000 L CNN
-F 1 "1uF" H 5265 5405 50  0000 L CNN
+F 1 "100nF" H 5265 5405 50  0000 L CNN
 F 2 "Capacitor_SMD:C_0805_2012Metric" H 5188 5300 50  0001 C CNN
 F 3 "~" H 5150 5450 50  0001 C CNN
@@
 P 4250 4900
 F 0 "D_boot1" V 4296 4820 50  0000 R CNN
-F 1 "D_Schottky" V 4205 4820 50  0000 R CNN
+F 1 "STTH4R02U" V 4205 4820 50  0000 R CNN
 F 2 "Diode_SMD:D_SMB" H 4250 4900 50  0001 C CNN
-F 3 "~" H 4250 4900 50  0001 C CNN
+F 3 "https://www.st.com/resource/en/datasheet/stth4r02.pdf" H 4250 4900 50  0001 C CNN
 	1    4250 4900
 	0    -1   -1   0
@@
 P 9700 4900
 F 0 "D_boot2" V 9746 4820 50  0000 R CNN
-F 1 "D_Schottky" V 9655 4820 50  0000 R CNN
+F 1 "STTH4R02U" V 9655 4820 50  0000 R CNN
 F 2 "Diode_SMD:D_SMB" H 9700 4900 50  0001 C CNN
-F 3 "~" H 9700 4900 50  0001 C CNN
+F 3 "https://www.st.com/resource/en/datasheet/stth4r02.pdf" H 9700 4900 50  0001 C CNN
 	1    9700 4900
 	0    -1   -1   0
@@
 Wire Wire Line
 	9700 5050 9700 5150
+$Comp
+L Device:R_Small R3
+U 1 1 5EA3727C
+P 2550 6300
+AR Path="/5EA3727C" Ref="R3"  Part="1"
+AR Path="/5E9944F3/5EA3727C" Ref="R5"  Part="1"
+F 0 "R3" H 2750 6400 50  0000 L CNN
+F 1 "20k" H 2750 6300 50  0000 L CNN
+F 2 "Resistor_SMD:R_0805_2012Metric" H 2550 6300 50  0001 C CNN
+F 3 "~" H 2550 6300 50  0001 C CNN
+	1    2550 6300
+	-1   0    0    1
+$EndComp
 $EndSCHEMATC

Commit message: Revision of the schematics - Part 1 of 3
The schematics of the measurement, driver and power parts were commented and reorganized.
Most of the work is focused on readeability. More detailed comments are to come.
Other:
- note added: "Driver stage inputs"
- note added: "Driver stage outputs"
- note added: "N/GND IGBT DRIVER"
- note added: "Synch. Boost Driver 1"
- note added: "Synch. Boost Driver 2"
- note added: "Synchronous Buck driver 1 consists of a boostrap driver.\nIt was implemented in accordance to the application note\nof the UCC21222DR component. \nIt's main features are resumed on the table below."
- note added: "Table to be filled..."
- note added: "The N/GND IGBT driver is composed of an optocoupler which \nis connected directly to the component's gate. \nSince the switching of this component is not made dynamically,\nits speed requirements are not critical and can be met with this\noptocoupler."
- note added: "These are the\ninputs for the \ndriver stage. \nThey are all \nlinked with \nthe measurement\nstage."
- note added: "These are the\ninputs for the \ndriver stage. \nThey are all\nlinked with \nthe power \nstage."
- moved on the sheet: C1, C10, C11, C12, C2, C3, C4, C5, C6, C7, C8, C9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
