File: KiCAD_files/Power.sch (KiCad schematic (older format))
At the start: 82 parts, among them J1 2604-1102, J2 2604-1102, J3 Power_Board_outline, J4 2604-1102, J5 2604-1102, Q1 QM6006D, Q2 QM6006D, Q3 Q_NIGBT_GCE, Q4 QM6006D, Q5 QM6006D, U1 ACS730xLCTR-20AB, U2 LM35-LP, U3 ACS712xLCTR-20A, U4 ACS730xLCTR-20AB

Commit message: Added missing values -references -  and datasheets to the power schematic.
Parts:
- D2, D3, D4, D5: value D -> STPS0520Z
- D_H1, D_H2, D_L1, D_L2: value D_Schottky_AKA -> STTH1002C
- F1, F2, F3, F4: value Polyfuse -> Polyfuse RKEF500
- Q1, Q2, Q4, Q5: value QM6006D -> IRFR4615
- Q3: value Q_NIGBT_GCE -> FGD3040G2-F085
- Rv1, Rv3: value R_Small -> 150K
- Rv2, Rv4: value R_Small -> 470
- Rv5: value R_Small -> 330K
- Rv6: value R_Small -> 5.6K

Commit message: Addded missing values and datasheet to measurment schematic Minor schematic modifications - added zener diodes
Changed lines of the file:
@@
 U 1 1 5E9DBBC2
 P 7100 4200
-F 0 "R_pdL1" H 7030 4154 50  0000 R CNN
-F 1 "1k" H 7030 4245 50  0000 R CNN
+F 0 "R_pdL1" H 7500 4150 50  0000 R CNN
+F 1 "1k" H 7350 4250 50  0000 R CNN
 F 2 "Resistor_SMD:R_0805_2012Metric" V 7030 4200 50  0001 C CNN
 F 3 "~" H 7100 4200 50  0001 C CNN
 	1    7100 4200
-	-1   0    0    1
-$EndComp
-$Comp
-L Device:R R_pdH1
-U 1 1 5E9DBBC9
-P 7100 3000
-F 0 "R_pdH1" H 7030 2954 50  0000 R CNN
-F 1 "1k" H 7030 3045 50  0000 R CNN
-F 2 "Resistor_SMD:R_0805_2012Metric" V 7030 3000 50  0001 C CNN
-F 3 "~" H 7100 3000 50  0001 C CNN
-	1    7100 3000
 	-1   0    0    1
 $EndComp
@@
 Text Label 9750 2100 0    50   ~ 0
 V_Out
-Text Label 3500 4300 0    50   ~ 0
-N
 Text Label 3500 4300 0    50   ~ 0
 N
@@
 U 1 1 5F4613E5
 P 4250 7350
-F 0 "C22" H 4342 7396 50  0000 L CNN
-F 1 "1nF" H 4342 7305 50  0000 L CNN
+F 0 "C22" H 3950 7450 50  0000 L CNN
+F 1 "1nF" H 3950 7350 50  0000 L CNN
 F 2 "Capacitor_SMD:C_0805_2012Metric" H 4250 7350 50  0001 C CNN
 F 3 "~" H 4250 7350 50  0001 C CNN
@@
 U 1 1 5E9DBC83
 P 4500 4100
-F 0 "C1" H 4592 4146 50  0000 L CNN
-F 1 "1nF" H 4592 4055 50  0000 L CNN
+F 0 "C1" H 4250 4150 50  0000 L CNN
+F 1 "1nF" H 4200 4050 50  0000 L CNN
 F 2 "Capacitor_SMD:C_0805_2012Metric" H 4500 4100 50  0001 C CNN
 F 3 "~" H 4500 4100 50  0001 C CNN
@@
 Text Label 3500 7550 0    50   ~ 0
 N
-Text Label 3500 7550 0    50   ~ 0
-N
 Wire Wire Line
 	2500 7200 2500 7550
@@
 U 1 1 5F461376
 P 7650 6150
-F 0 "R_pdH2" H 7580 6104 50  0000 R CNN
-F 1 "1k" H 7580 6195 50  0000 R CNN
+F 0 "R_pdH2" H 8050 6100 50  0000 R CNN
+F 1 "1k" H 7850 6200 50  0000 R CNN
 F 2 "Resistor_SMD:R_0805_2012Metric" V 7580 6150 50  0001 C CNN
 F 3 "~" H 7650 6150 50  0001 C CNN
@@
 U 1 1 5F461370
 P 7650 7350
-F 0 "R_pdL2" H 7580 7304 50  0000 R CNN
-F 1 "1k" H 7580 7395 50  0000 R CNN
+F 0 "R_pdL2" H 8050 7300 50  0000 R CNN
+F 1 "1k" H 7850 7400 50  0000 R CNN
 F 2 "Resistor_SMD:R_0805_2012Metric" V 7580 7350 50  0001 C CNN
 F 3 "~" H 7650 7350 50  0001 C CNN
@@
 	0    1    1    0
 $EndComp
+$Comp
+L Device:R R_pdH1
+U 1 1 5E9DBBC9
+P 7100 3000
+F 0 "R_pdH1" H 7450 2950 50  0000 R CNN
+F 1 "1k" H 7300 3050 50  0000 R CNN
+F 2 "Resistor_SMD:R_0805_2012Metric" V 7030 3000 50  0001 C CNN
+F 3 "~" H 7100 3000 50  0001 C CNN
+	1    7100 3000
+	-1   0    0    1
+$EndComp
 $EndSCHEMATC

Commit message: Revision of the schematics - Part 1 of 3
The schematics of the measurement, driver and power parts were commented and reorganized.
Most of the work is focused on readeability. More detailed comments are to come.
Other:
- note added: "DO NOT FORGET!"
- note added: "NEUTRAL TO GROUND\nCONNECTION"
Changed lines of the file:
@@
 Text Label 14950 2650 0    50   ~ 0
 IIHigh
-Text Label 3900 9500 0    50   ~ 0
+Text Label 3810 10670 0    50   ~ 0
 VTh
 Text Label 9750 2100 0    50   ~ 0
@@
 Text Label 5600 4350 0    50   ~ 0
 DGND
-Text Label 3350 9900 0    50   ~ 0
+Text Label 3260 11070 0    50   ~ 0
 DGND
 Wire Wire Line
-	3350 9800 3350 9900
-Text Label 4000 8450 0    50   ~ 0
+	3260 10970 3260 11070
+Text Label 4050 9050 0    50   ~ 0
 N
 Wire Wire Line
-	4000 8450 3700 8450
+	4050 9050 3750 9050
 $Comp
 L power:GNDREF #PWR02
 U 1 1 5EBD4EE3
-P 3950 8950
-F 0 "#PWR02" H 3950 8700 50  0001 C CNN
-F 1 "GNDREF" H 3955 8777 50  0000 C CNN
-F 2 "" H 3950 8950 50  0001 C CNN
-F 3 "" H 3950 8950 50  0001 C CNN
-	1    3950 8950
+P 4000 9550
+F 0 "#PWR02" H 4000 9300 50  0001 C CNN
+F 1 "GNDREF" H 4005 9377 50  0000 C CNN
+F 2 "" H 4000 9550 50  0001 C CNN
+F 3 "" H 4000 9550 50  0001 C CNN
+	1    4000 9550
 	0    -1   -1   0
 $EndComp
-Text Label 2650 8650 0    50   ~ 0
+Text Label 2700 9250 0    50   ~ 0
 Neutral_GND_cmd
 Wire Wire Line
-	2650 8650 3400 8650
-Wire Wire Line
-	3700 8850 3700 8950
-Wire Wire Line
-	3700 8950 3950 8950
+	2700 9250 3450 9250
+Wire Wire Line
+	3750 9450 3750 9550
+Wire Wire Line
+	3750 9550 4000 9550
 $Comp
 L Device:Q_NIGBT_GCE Q3
 U 1 1 5EC2B2E3
-P 3600 8650
-F 0 "Q3" H 3790 8696 50  0000 L CNN
-F 1 "FGD3040G2-F085" H 3790 8605 50  0000 L CNN
-F 2 "Package_TO_SOT_SMD:TO-252-2" H 3800 8750 50  0001 C CNN
-F 3 "https://www.onsemi.com/pub/Collateral/FGI3040G2_F085-D.PDF" H 3600 8650 50  0001 C CNN
-	1    3600 8650
+P 3650 9250
+F 0 "Q3" H 3840 9296 50  0000 L CNN
+F 1 "FGD3040G2-F085" H 3840 9205 50  0000 L CNN
+F 2 "Package_TO_SOT_SMD:TO-252-2" H 3850 9350 50  0001 C CNN
+F 3 "https://www.onsemi.com/pub/Collateral/FGI3040G2_F085-D.PDF" H 3650 9250 50  0001 C CNN
+	1    3650 9250
 	1    0    0    -1
 $EndComp
@@
 	15450 2100 15450 3050
 Wire Wire Line
-	3750 9500 3900 9500
+	3660 10670 3810 10670
 Connection ~ 3500 3700
 Wire Wire Line
@@
 	13800 4150 14200 4150
 Wire Wire Line
-	650  2150 1550 2150
-Wire Wire Line
-	650  5300 1550 5300
+	1090 2150 1550 2150
+Wire Wire Line
+	1090 5300 1550 5300
 Wire Wire Line
 	4500 4000 4500 3900
@@
 	2150 4000 2150 4100
 Wire Wire Line
-	650  2150 650  3250
+	1090 2150 1090 3250
 $Comp
 L Symbols:2604-1102 J1
 U 1 1 5F36DFF1
-P 1050 3450
-F 0 "J1" H 1178 3553 60  0000 L CNN
-F 1 "2604-1102" H 1178 3447 60  0000 L CNN
-F 2 "Footprints:WAGO-2604-1102" H 1050 3390 60  0001 C CNN
-F 3 "" H 1050 3450 60  0000 C CNN
-	1    1050 3450
-	1    0    0    -1
+P 690 3450
+F 0 "J1" H 630 3820 60  0000 L CNN
+F 1 "2604-1102" H 350 3930 60  0000 L CNN
+F 2 "Footprints:WAGO-2604-1102" H 690 3390 60  0001 C CNN
+F 3 "" H 690 3450 60  0000 C CNN
+	1    690  3450
+	-1   0    0    -1
 $EndComp
 $Comp
@@
 U 1 1 5F370ABD
 P 1750 4100
-F 0 "J2" H 1878 4203 60  0000 L CNN
-F 1 "2604-1102" H 1878 4097 60  0000 L CNN
+F 0 "J2" H 1700 3850 60  0000 L CNN
+F 1 "2604-1102" H 1480 3760 60  0000 L CNN
 F 2 "Footprints:WAGO-2604-1102" H 1750 4040 60  0001 C CNN
 F 3 "" H 1750 4100 60  0000 C CNN
@@
 $EndComp
 Wire Wire Line
-	650  3350 650  3250
-Connection ~ 650  3250
-Wire Wire Line
-	650  3450 650  3550
-Connection ~ 650  3550
-Wire Wire Line
-	650  3550 650  5300
+	1090 3350 1090 3250
+Connection ~ 1090 3250
+Wire Wire Line
+	1090 3450 1090 3550
+Connection ~ 1090 3550
+Wire Wire Line
+	1090 3550 1090 5300
 Wire Wire Line
 	14200 3850 14200 3950
@@
 L power:+5VD #PWR0106
 U 1 1 5F3D4930
-P 3350 9150
-F 0 "#PWR0106" H 3350 9000 50  0001 C CNN
-F 1 "+5VD" H 3365 9323 50  0000 C CNN
-F 2 "" H 3350 9150 50  0001 C CNN
-F 3 "" H 3350 9150 50  0001 C CNN
-	1    3350 9150
-	1    0    0    -1
-$EndComp
-Wire Wire Line
-	3350 9200 3350 9150
+P 3260 10320
+F 0 "#PWR0106" H 3260 10170 50  0001 C CNN
+F 1 "+5VD" H 3275 10493 50  0000 C CNN
+F 2 "" H 3260 10320 50  0001 C CNN
+F 3 "" H 3260 10320 50  0001 C CNN
+	1    3260 10320
+	1    0    0    -1
+$EndComp
+Wire Wire Line
+	3260 10370 3260 10320
 $Comp
 L power:+5VD #PWR0110
@@
 L Sensor_Temperature:LM35-LP U2
 U 1 1 5F342246
-P 3350 9500
-F 0 "U2" H 3021 9546 50  0000 R CNN
-F 1 "LM35-LP" H 3021 9455 50  0000 R CNN
-F 2 "Package_TO_SOT_THT:TO-92" H 3400 9250 50  0001 L CNN
-F 3 "http://www.ti.com/lit/ds/symlink/lm35.pdf" H 3350 9500 50  0001 C CNN
-	1    3350 9500
+P 3260 10670
+F 0 "U2" H 2931 10716 50  0000 R CNN
+F 1 "LM35-LP" H 2931 10625 50  0000 R CNN
+F 2 "Package_TO_SOT_THT:TO-92" H 3310 10420 50  0001 L CNN
+F 3 "http://www.ti.com/lit/ds/symlink/lm35.pdf" H 3260 10670 50  0001 C CNN
+	1    3260 10670
 	1    0    0    -1
 $EndComp
@@
 	-1   0    0    1
 $EndComp
+Wire Notes Line
+	4750 3970 4750 4650
+Wire Notes Line
+	4750 4650 3740 4650
+Wire Notes Line
+	3740 4650 3740 3970
+Wire Notes Line
+	3740 3970 4750 3970
+Text Notes 3740 4570 0    79   ~ 16
+DO NOT FORGET!
+Text Notes 590  9310 0    197  ~ 39
+NEUTRAL TO GROUND\nCONNECTION
 $EndSCHEMATC
