File: KiCAD_files/Power.sch (KiCad schematic (older format))
At the start: 170 parts, among them J1 2604-1102, J10 Conn_01x01, J11 Conn_01x01, J12 Conn_01x01, J13 Conn_01x01, J14 Conn_01x01, J15 Conn_01x01, J16 Conn_01x01, J17 Conn_01x01, J18 Conn_01x01, J19 Conn_01x01, J2 2604-1102, J20 Conn_01x01, J21 Conn_01x01, J22 Conn_01x01, J23 Conn_01x01, J24 Conn_01x01, J25 Conn_01x01, J26 Conn_01x01, J27 Conn_01x01, J28 Conn_01x01, J29 Conn_01x01, J3 Conn_01x01, J30 Conn_01x01, J31 Conn_01x01, J32 Conn_01x01, J33 Conn_01x01, J34 Conn_01x01, J35 Conn_01x01, J4 2604-1102, J5 2604-1102, J6 Conn_01x01, J7 Conn_01x01, J8 Conn_01x01, J9 Conn_01x01, Q1 IPD200N15N3, Q2 IPD200N15N3, Q3 IPD200N15N3, Q4 IPD200N15N3, Q5 IPD200N15N3, U1 ACS730xLCTR-20AB, U10 OPA316, U11 OPA316, U12 OPA316, U13 OPA316, U3 ACS712xLCTR-20A, U4 ACS730xLCTR-20AB, U5 AMC1311, U6 AMC1100DUB, U7 AMC1100DUB, U8 OPA316, U9 OPA316

Commit message: WIP: Layout test V1.1.3
Parts:
- removed JP1, JP10, JP2, JP3, JP4, JP5, JP6, JP7, JP8, JP9: THJP0612AST, Resistor_SMD:R_0612_1632Metric, symbol Device:Jumper_NO_Small
- added C39, C40, C41, C42: 100nF, Capacitor_SMD:C_1210_3225Metric, symbol Device:C
- added J36: 2604-1102, Footprints:WAGO-2604-1102, symbol Symbols:2604-1102
- D_H1, D_H2, D_L1, D_L2: footprint Package_TO_SOT_SMD:TO-252-2 -> Diode_SMD:D_SOD-123
Connections:
- net labels added: Earth_Protective
- wire segments 528 -> 517
Other:
- moved on the sheet: C11, C12, HS1, J1

Commit message: Added the third power leg. Changed the unductor to 33uH SRP1510. Started a draft of power layout
Parts:
- removed Cs3: C_Small, Capacitor_SMD:C_0805_2012Metric, symbol Device:C_Small
- removed D_H1, D_H2: STTH1002CB, Diode_SMD:D_SOD-123, symbol Device:D_Schottky_AKA
- removed Rs3: R_Small, Resistor_SMD:R_0805_2012Metric, symbol Device:R_Small
- added C43, C44, C45: 4.7uF, Capacitor_SMD:C_1210_3225Metric, symbol Device:C
- added C46: 1nF, Capacitor_SMD:C_0805_2012Metric, symbol Device:C_Small
- added C47, C51, C52, C53, C54: 100nF, Capacitor_SMD:C_0805_2012Metric, symbol Device:C_Small
- added C48, C49, C50: 100nF, Capacitor_SMD:C_1210_3225Metric, symbol Device:C
- added D1, D6: STPS0520Z, Diode_SMD:D_SOD-123, symbol Device:D
- added D_L3: STTH1002CB, Diode_SMD:D_SOD-123, symbol Device:D_Schottky_AKA
- added F5: Nano2 fuse holder, Footprints:Fuse_holder_omni_blok, symbol Device:Fuse
- added J37: 2604-1102, Footprints:WAGO-2604-1102, symbol Symbols:2604-1102
- added J38, J39, J40, J41, J42, J43, J44, J45: Conn_01x01, Footprints:0906_millmax, symbol Connector_Generic:Conn_01x01
- added L3: 33uH, Footprints:SRP1510CA-330M, symbol pspice:INDUCTOR
- added Q6, Q7: IPD200N15N3, Package_TO_SOT_SMD:TO-252-2, symbol Transistor_FET:QM6006D
- added R37, R38: 2,2, Resistor_SMD:R_0805_2012Metric, symbol Device:R
- added R39, R40: 0, Resistor_SMD:R_0805_2012Metric, symbol Device:R
- added R41, R42: 1k, Resistor_SMD:R_0805_2012Metric, symbol Device:R
- added R43, R44: 27k, Resistor_SMD:R_0805_2012Metric, symbol Device:R_Small
- added R45, R46: 12k, Resistor_SMD:R_0805_2012Metric, symbol Device:R_Small
- added R47, R48: 200k, Resistor_SMD:R_0805_2012Metric, symbol Device:R_Small
- added R49, R50: 82k, Resistor_SMD:R_0805_2012Metric, symbol Device:R_Small
- added Rv7: 150K, Resistor_SMD:R_0805_2012Metric, symbol Device:R_Small
- added Rv8: 470, Resistor_SMD:R_0805_2012Metric, symbol Device:R_Small
- added U14: AMC1100DUB, Footprints:SOP-8_6.62x9.15mm_P2.54mm, symbol Symbols:AMC1100
- added U15, U16: OPA316, Package_TO_SOT_SMD:SOT-353_SC-70-5, symbol Amplifier_Operational:TLV6001DCK
- added U2: ACS730xLCTR-20AB, Package_SO:SOIC-8_3.9x4.9mm_P1.27mm, symbol Sensor_Current:ACS730xLCTR-20AB
- L1, L2: value 47uH -> 33uH; footprint Footprints:WE-HCF-2013 -> Footprints:SRP1510CA-330M; manf# 7443634700 -> SRP1510CA-330M
Connections:
- net +5V: now also C51.1, U14.1 (VDD1)
- net +5VD: now also C47.2, C52.1, C53.1, C54.1, U14.8 (VDD2), U15.5 (V+), U16.5 (V+), U2.8 (VCC)
- net DGND: now also C46.1, C47.1, C52.2, C53.2, C54.2, J43.1 (Pin_1), J45.1 (Pin_1), R48.1, R49.2, U14.5 (GND2), U15.2 (V-), U16.2 (V-), U2.5 (GND)
- net GNDREF: now also Cs1.2, C48.2, C49.2, C50.2, D_L3.1 (A), D_L3.3 (A), J41.1 (Pin_1), Q7.3 (S), R42.1
- net N: now also C43.2, C44.2, C45.2, C51.2, Rv8.2, U14.3 (VINN), U14.4 (GND1)
- net PWM_H2: now also D1.1 (K), R37.1
- net SW_Node1: no longer Cs1.2
- net V_Out: now also C48.1, C49.1, C50.1, Q6.2 (D); no longer Rs1.1
- net Vref: now also R45.1
- new net: D1.2 (A), R39.1
- new net: Q6.1 (G), R37.2, R39.2, R41.2
- new net: Q7.1 (G), R38.2, R40.2, R42.2
- new net: D6.1 (K), R38.1
- new net: D6.2 (A), R40.1
- new net: L3.1, U2.1 (IP+), U2.2 (IP+)
- new net: C46.2, U2.6 (VZCR)
- new net: F5.2, J37.1, J37.2, J37.3, J37.4
- new net: R44.1, U14.6 (VOUTN)
- new net: R43.1, U14.7 (VOUTP)
- new net: R43.2, R45.2, U15.1 (+)
- new net: R44.2, R46.1, U15.3 (-)
- new net: R48.2, R50.1, U16.3 (-)
- new net: R47.2, R49.1, U16.1 (+)
- new net IILow3: R47.1, U2.7 (VIOUT)
- new net IILow3_op: J44.1 (Pin_1), R50.2, U16.4
- new net PWM_H3: J38.1 (Pin_1)
- new net PWM_L3: J40.1 (Pin_1)
- new net SW_Node3: D_L3.2 (K), J39.1 (Pin_1), L3.2, Q6.3 (S), Q7.2 (D), R41.1, Rs1.1
- new net VILow3+: Rv7.2, Rv8.1, U14.2 (VINP)
- new net VILow3_op: J42.1 (Pin_1), R46.2, U15.4
- new net VI_LOW3: C43.1, C44.1, C45.1, F5.1, Rv7.1, U2.3 (IP-), U2.4 (IP-)
Other:
- moved on the sheet: C1, C10, C11, C12, C13, C14, C15, C16, C17, C18, C19, C2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

Commit message: Rearranged the schematic for a 3 leg version using subsheets.
Parts:
- C11, C12, C39, C40, C48, C49: footprint Capacitor_SMD:C_1210_3225Metric -> Capacitor_SMD:C_0805_2012Metric
Changed lines of the file:
@@
 F 0 "C11" H 9515 6471 50  0000 L CNN
 F 1 "100nF" H 9515 6380 50  0000 L CNN
-F 2 "Capacitor_SMD:C_1210_3225Metric" H 9438 6275 50  0001 C CNN
+F 2 "Capacitor_SMD:C_0805_2012Metric" H 9438 6275 50  0001 C CNN
 F 3 "~" H 9400 6425 50  0001 C CNN
 F 4 "1210PC104KAT1A" H 9400 6425 50  0001 C CNN "manf#"
@@
 F 0 "C12" H 9515 9721 50  0000 L CNN
 F 1 "100nF" H 9515 9630 50  0000 L CNN
-F 2 "Capacitor_SMD:C_1210_3225Metric" H 9438 9525 50  0001 C CNN
+F 2 "Capacitor_SMD:C_0805_2012Metric" H 9438 9525 50  0001 C CNN
 F 3 "~" H 9400 9675 50  0001 C CNN
 F 4 "1210PC104KAT1A" H 9400 9675 50  0001 C CNN "manf#"
@@
 F 0 "C40" H 9965 6471 50  0000 L CNN
 F 1 "100nF" H 9965 6380 50  0000 L CNN
-F 2 "Capacitor_SMD:C_1210_3225Metric" H 9888 6275 50  0001 C CNN
+F 2 "Capacitor_SMD:C_0805_2012Metric" H 9888 6275 50  0001 C CNN
 F 3 "~" H 9850 6425 50  0001 C CNN
 F 4 "1210PC104KAT1A" H 9850 6425 50  0001 C CNN "manf#"
@@
 F 0 "C39" H 9990 9721 50  0000 L CNN
 F 1 "100nF" H 9990 9630 50  0000 L CNN
-F 2 "Capacitor_SMD:C_1210_3225Metric" H 9913 9525 50  0001 C CNN
+F 2 "Capacitor_SMD:C_0805_2012Metric" H 9913 9525 50  0001 C CNN
 F 3 "~" H 9875 9675 50  0001 C CNN
 F 4 "1210PC104KAT1A" H 9875 9675 50  0001 C CNN "manf#"
@@
 F 0 "C48" H 9465 12921 50  0000 L CNN
 F 1 "100nF" H 9465 12830 50  0000 L CNN
-F 2 "Capacitor_SMD:C_1210_3225Metric" H 9388 12725 50  0001 C CNN
+F 2 "Capacitor_SMD:C_0805_2012Metric" H 9388 12725 50  0001 C CNN
 F 3 "~" H 9350 12875 50  0001 C CNN
 F 4 "1210PC104KAT1A" H 9350 12875 50  0001 C CNN "manf#"
@@
 F 0 "C49" H 9940 12921 50  0000 L CNN
 F 1 "100nF" H 9940 12830 50  0000 L CNN
-F 2 "Capacitor_SMD:C_1210_3225Metric" H 9863 12725 50  0001 C CNN
+F 2 "Capacitor_SMD:C_0805_2012Metric" H 9863 12725 50  0001 C CNN
 F 3 "~" H 9825 12875 50  0001 C CNN
 F 4 "1210PC104KAT1A" H 9825 12875 50  0001 C CNN "manf#"
