File: KiCAD_files/_autosave-Power.sch (KiCad schematic (older format))
At the start: 82 parts, among them J1 2604-1102, J2 2604-1102, J3 Power_Board_outline, J4 2604-1102, J5 2604-1102, Q1 IRFR4615, Q2 IRFR4615, Q3 FGD3040G2-F085, Q4 IRFR4615, Q5 IRFR4615, U1 ACS730xLCTR-20AB, U2 LM35-LP, U3 ACS712xLCTR-20A, U4 ACS730xLCTR-20AB

Commit message: Modifications on the power part
Some changes were made to the power schematics. There are still some nets to be highlighted and so forth.
Connections:
- wire segments 346 -> 347
Other:
- note added: "T\nSensors"
- moved on the sheet: C4, C5, Rv5, Rv6
Changed lines of the file:
@@
 	15250 4850 15150 4850
 Wire Wire Line
-	8420 9810 8420 10260
-Text Label 8420 9960 0    50   ~ 0
+	8010 9900 8010 10350
+Text Label 8010 10050 0    50   ~ 0
 VIHigh-
 $Comp
 L Device:R_Small Rv6
 U 1 1 5F5D7CCC
-P 8420 9710
-F 0 "Rv6" H 8479 9756 50  0000 L CNN
-F 1 "5.6K" H 8479 9665 50  0000 L CNN
-F 2 "Resistor_SMD:R_0805_2012Metric" H 8420 9710 50  0001 C CNN
-F 3 "~" H 8420 9710 50  0001 C CNN
-	1    8420 9710
-	1    0    0    -1
-$EndComp
-Text Label 8420 9510 0    50   ~ 0
+P 8010 9800
+F 0 "Rv6" H 8069 9846 50  0000 L CNN
+F 1 "5.6K" H 8069 9755 50  0000 L CNN
+F 2 "Resistor_SMD:R_0805_2012Metric" H 8010 9800 50  0001 C CNN
+F 3 "~" H 8010 9800 50  0001 C CNN
+	1    8010 9800
+	1    0    0    -1
+$EndComp
+Text Label 8010 9600 0    50   ~ 0
 VIHigh+
 Wire Wire Line
-	8420 9360 8420 9610
+	8010 9450 8010 9700
 $Comp
 L Device:R_Small Rv5
 U 1 1 5F5D7CC2
-P 8420 9260
-F 0 "Rv5" H 8479 9306 50  0000 L CNN
-F 1 "330K" H 8479 9215 50  0000 L CNN
-F 2 "Resistor_SMD:R_0805_2012Metric" H 8420 9260 50  0001 C CNN
-F 3 "~" H 8420 9260 50  0001 C CNN
-	1    8420 9260
+P 8010 9350
+F 0 "Rv5" H 8069 9396 50  0000 L CNN
+F 1 "330K" H 8069 9305 50  0000 L CNN
+F 2 "Resistor_SMD:R_0805_2012Metric" H 8010 9350 50  0001 C CNN
+F 3 "~" H 8010 9350 50  0001 C CNN
+	1    8010 9350
 	1    0    0    -1
 $EndComp
@@
 	4490 10340 4890 10340
 Wire Wire Line
-	8420 10260 8630 10260
+	8010 10350 8220 10350
 Text Label 14000 2560 2    50   ~ 0
 N
@@
 Wire Wire Line
 	8410 6040 8410 6090
-Text Label 11130 5190 2    50   ~ 0
+Text Label 12360 4570 2    197  ~ 39
 V_Out
 $Comp
@@
 L power:GNDREF #PWR?
 U 1 1 5F749262
-P 8630 10370
+P 8220 10460
 AR Path="/5E91AAF4/5F749262" Ref="#PWR?"  Part="1"
 AR Path="/5E86B783/5F749262" Ref="#PWR?"  Part="1"
 AR Path="/5E99427A/5F749262" Ref="#PWR?"  Part="1"
 AR Path="/5F749262" Ref="#PWR?"  Part="1"
-F 0 "#PWR?" H 8630 10120 50  0001 C CNN
-F 1 "GNDREF" H 8635 10197 50  0000 C CNN
-F 2 "" H 8630 10370 50  0001 C CNN
-F 3 "" H 8630 10370 50  0001 C CNN
-	1    8630 10370
-	1    0    0    -1
-$EndComp
-Wire Wire Line
-	8630 10370 8630 10260
+F 0 "#PWR?" H 8220 10210 50  0001 C CNN
+F 1 "GNDREF" H 8225 10287 50  0000 C CNN
+F 2 "" H 8220 10460 50  0001 C CNN
+F 3 "" H 8220 10460 50  0001 C CNN
+	1    8220 10460
+	1    0    0    -1
+$EndComp
+Wire Wire Line
+	8220 10460 8220 10350
 Connection ~ 10370 2450
 Text Label 3470 8850 2    50   ~ 0
 V_Out
-Text Label 5960 8950 0    50   ~ 0
-V_Out
 $Comp
 L power:+5VD #PWR0110
 U 1 1 5F406701
-P 7780 9400
-F 0 "#PWR0110" H 7780 9250 50  0001 C CNN
-F 1 "+5VD" H 7795 9573 50  0000 C CNN
-F 2 "" H 7780 9400 50  0001 C CNN
-F 3 "" H 7780 9400 50  0001 C CNN
-	1    7780 9400
+P 6940 9490
+F 0 "#PWR0110" H 6940 9340 50  0001 C CNN
+F 1 "+5VD" H 6955 9663 50  0000 C CNN
+F 2 "" H 6940 9490 50  0001 C CNN
+F 3 "" H 6940 9490 50  0001 C CNN
+	1    6940 9490
 	-1   0    0    -1
 $EndComp
@@
 L Device:C_Small C4
 U 1 1 5E9DBC6A
-P 7640 9910
-F 0 "C4" H 7520 10000 50  0000 L CNN
-F 1 "100nF" H 7360 9810 50  0000 L CNN
-F 2 "Capacitor_SMD:C_0805_2012Metric" H 7640 9910 50  0001 C CNN
-F 3 "~" H 7640 9910 50  0001 C CNN
-	1    7640 9910
+P 6800 10000
+F 0 "C4" H 6680 10090 50  0000 L CNN
+F 1 "100nF" H 6520 9900 50  0000 L CNN
+F 2 "Capacitor_SMD:C_0805_2012Metric" H 6800 10000 50  0001 C CNN
+F 3 "~" H 6800 10000 50  0001 C CNN
+	1    6800 10000
 	-1   0    0    -1
 $EndComp
-Text Label 6900 10640 2    50   ~ 0
+Text Label 6060 10730 2    50   ~ 0
 DGND
-Text Label 7360 10280 2    50   ~ 0
+Text Label 6520 10370 2    50   ~ 0
 IIHigh
 Wire Wire Line
-	7130 9930 7130 10280
+	6290 10020 6290 10370
 $Comp
 L Device:C_Small C5
 U 1 1 5E9DBC8A
-P 6900 10250
-F 0 "C5" H 6992 10296 50  0000 L CNN
-F 1 "1nF" H 6992 10205 50  0000 L CNN
-F 2 "Capacitor_SMD:C_0805_2012Metric" H 6900 10250 50  0001 C CNN
-F 3 "~" H 6900 10250 50  0001 C CNN
-	1    6900 10250
+P 6060 10340
+F 0 "C5" H 6152 10386 50  0000 L CNN
+F 1 "1nF" H 6152 10295 50  0000 L CNN
+F 2 "Capacitor_SMD:C_0805_2012Metric" H 6060 10340 50  0001 C CNN
+F 3 "~" H 6060 10340 50  0001 C CNN
+	1    6060 10340
 	-1   0    0    -1
 $EndComp
 Wire Wire Line
-	6730 9530 6580 9530
+	5890 9620 5740 9620
 $Comp
 L Sensor_Current:ACS712xLCTR-20A U3
 U 1 1 5E9DBC38
-P 7130 9530
-F 0 "U3" V 6880 9940 50  0000 C CNN
-F 1 "ACS712xLCTR-20A" V 6750 10180 50  0000 C CNN
-F 2 "Package_SO:SOIC-8_3.9x4.9mm_P1.27mm" H 7230 9180 50  0001 L CIN
-F 3 "http://www.allegromicro.com/~/media/Files/Datasheets/ACS712-Datasheet.ashx?la=en" H 7130 9530 50  0001 C CNN
-	1    7130 9530
+P 6290 9620
+F 0 "U3" V 6040 10030 50  0000 C CNN
+F 1 "ACS712xLCTR-20A" V 5910 10270 50  0000 C CNN
+F 2 "Package_SO:SOIC-8_3.9x4.9mm_P1.27mm" H 6390 9270 50  0001 L CIN
+F 3 "http://www.allegromicro.com/~/media/Files/Datasheets/ACS712-Datasheet.ashx?la=en" H 6290 9620 50  0001 C CNN
+	1    6290 9620
 	0    1    1    0
 $EndComp
 Wire Wire Line
-	7030 9930 6900 9930
-Wire Wire Line
-	6900 9930 6900 10150
-Text Label 7860 10290 2    50   ~ 0
+	6190 10020 6060 10020
+Wire Wire Line
+	6060 10020 6060 10240
+Text Label 7020 10380 2    50   ~ 0
 DGND
 Wire Wire Line
-	7640 10010 7640 10290
-Wire Wire Line
-	7640 10290 7860 10290
-Wire Wire Line
-	6580 9530 6580 10470
-Wire Wire Line
-	6580 10470 6670 10470
-Wire Wire Line
-	6900 10470 6900 10350
-Wire Wire Line
-	6900 10640 6670 10640
-Wire Wire Line
-	6670 10640 6670 10470
-Connection ~ 6670 10470
-Wire Wire Line
-	6670 10470 6900 10470
-Wire Wire Line
-	7130 10280 7360 10280
-Wire Wire Line
-	7530 9530 7640 9530
-Wire Wire Line
-	7780 9530 7780 9400
-Wire Wire Line
-	7640 9810 7640 9530
-Connection ~ 7640 9530
-Wire Wire Line
-	7640 9530 7780 9530
-Wire Wire Line
-	6930 8950 6930 9130
-Wire Wire Line
-	5960 8950 6930 8950
-Wire Wire Line
-	7330 9130 7330 8940
-Wire Wire Line
-	7330 8940 8420 8940
-Wire Wire Line
-	8420 9160 8420 8940
+	6800 10100 6800 10380
+Wire Wire Line
+	6800 10380 7450 10380
+Wire Wire Line
+	5740 9620 5740 10560
+Wire Wire Line
+	5740 10560 5830 10560
+Wire Wire Line
+	6060 10560 6060 10440
+Wire Wire Line
+	6060 10730 5830 10730
+Wire Wire Line
+	5830 10730 5830 10560
+Connection ~ 5830 10560
+Wire Wire Line
+	5830 10560 6060 10560
+Wire Wire Line
+	6290 10370 6520 10370
+Wire Wire Line
+	6690 9620 6800 9620
+Wire Wire Line
+	6940 9620 6940 9490
+Wire Wire Line
+	6800 9900 6800 9620
+Connection ~ 6800 9620
+Wire Wire Line
+	6800 9620 6940 9620
+Wire Wire Line
+	6090 9040 6090 9220
+Wire Wire Line
+	6490 9220 6490 9030
+Wire Wire Line
+	6490 9030 8010 9030
+Wire Wire Line
+	8010 9250 8010 9030
 Connection ~ 14810 1310
 Wire Wire Line
@@
 Wire Wire Line
 	13790 1200 13790 1150
-Text Label 14190 1200 2    50   ~ 0
+Text Label 14190 1010 2    98   ~ 20
 I_Low+_1
 Wire Wire Line
@@
 Wire Wire Line
 	13790 1400 13790 1450
-Text Label 14200 1400 2    50   ~ 0
+Text Label 14200 1400 2    50   ~ 10
 I_Low+_2
 Wire Wire Line
@@
 Wire Wire Line
 	14800 2390 14800 2440
-Text Label 8740 8940 2    50   ~ 0
+Text Label 8330 9030 2    50   ~ 0
 V_High+
 Wire Wire Line
-	8420 8940 8740 8940
-Connection ~ 8420 8940
+	8010 9030 8330 9030
+Connection ~ 8010 9030
 Wire Wire Line
 	14430 1310 14810 1310
@@
 Balancing\nResistors
 Wire Notes Line
-	7840 8840 8210 8840
-Wire Notes Line
-	8210 8840 8210 10830
-Text Notes 7820 8820 0    50   ~ 10
+	7430 8930 7800 8930
+Wire Notes Line
+	7800 8930 7800 10920
+Text Notes 7230 8900 0    50   ~ 10
 Output\ncurrent sensor
 Wire Notes Line
-	8460 8840 8830 8840
-Wire Notes Line
-	8830 8840 8830 10830
-Text Notes 8440 8820 0    50   ~ 10
+	8050 8930 8420 8930
+Wire Notes Line
+	8420 8930 8420 10920
+Text Notes 8030 8910 0    50   ~ 10
 Output \nVoltage sensor
 Text Notes 590  880  0    197  ~ 39
@@
 	14550 6830 14960 6830
 Wire Notes Line
-	14960 6830 14960 6530
-Wire Notes Line
 	14960 6530 14550 6530
 Text Notes 14560 6710 0    50   ~ 10
@@
 Wire Notes Line
 	11240 5050 11240 7260
+Wire Notes Line
+	14760 6750 14760 7010
+Wire Notes Line
+	14760 7010 14960 7010
+Wire Notes Line
+	14960 6740 14760 6740
+Wire Notes Line
+	14960 6530 14960 7010
+Text Notes 14770 7000 0    50   ~ 10
+T\nSensors
+Wire Notes Line
+	11830 5900 11830 610
+Wire Notes Line
+	11830 610  11840 610
+Wire Wire Line
+	4890 9040 6090 9040
+Connection ~ 4890 9040
+Wire Wire Line
+	14190 1200 14190 1010
 $EndSCHEMATC
