File: KiCAD_files/Measurment.sch (KiCad schematic (older format))
At the start: 66 parts, among them J1 Measurment_stage_outline_outp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, J2 Measurment_stage_outline_sign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, J3 Conn_01x02, U1 NMA1505SC, U2 AMC1100, U3 AMC1100, U4 AMC1311, U5 R-78C5.0-1.0, U6 AMS1117-3.3, U7 NMA1505SC

Commit message: Added missing 3Dfootprints
Parts:
- U2, U3, U4: footprint Package_SO:SOIC-8_7.5x5.85mm_P1.27mm -> Footprints:SOIC-8_7.5x5.85mm_P1.27mm
Changed lines of the file:
@@
 F 0 "U2" H 4500 2365 50  0000 C CNN
 F 1 "AMC1100" H 4500 2274 50  0000 C CNN
-F 2 "Package_SO:SOIC-8_7.5x5.85mm_P1.27mm" H 4500 1450 50  0001 C CNN
+F 2 "Footprints:SOIC-8_7.5x5.85mm_P1.27mm" H 4500 1450 50  0001 C CNN
 F 3 "https://www.ti.com/lit/ds/symlink/amc1100.pdf?ts=1597048467257&ref_url=https%253A%252F%252Fwww.google.com%252F" H 4500 1450 50  0001 C CNN
 	1    4500 1700
@@
 F 0 "U3" H 4500 3615 50  0000 C CNN
 F 1 "AMC1100" H 4500 3524 50  0000 C CNN
-F 2 "Package_SO:SOIC-8_7.5x5.85mm_P1.27mm" H 4500 2700 50  0001 C CNN
+F 2 "Footprints:SOIC-8_7.5x5.85mm_P1.27mm" H 4500 2700 50  0001 C CNN
 F 3 "https://www.ti.com/lit/ds/symlink/amc1100.pdf?ts=1597048467257&ref_url=https%253A%252F%252Fwww.google.com%252F" H 4500 2700 50  0001 C CNN
 	1    4500 2950
@@
 F 0 "U4" H 4500 5315 50  0000 C CNN
 F 1 "AMC1311" H 4500 5224 50  0000 C CNN
-F 2 "Package_SO:SOIC-8_7.5x5.85mm_P1.27mm" H 4500 4400 50  0001 C CNN
+F 2 "Footprints:SOIC-8_7.5x5.85mm_P1.27mm" H 4500 4400 50  0001 C CNN
 F 3 "https://www.ti.com/lit/ds/symlink/amc1311.pdf?ts=1597049043074&ref_url=https%253A%252F%252Fwww.google.com%252F" H 4500 4400 50  0001 C CNN
 	1    4500 4650
