File: KiCAD_files/Power.kicad_pcb (KiCad board)
At the start: 4 copper layers, 100 x 100 mm, 169 parts, among them J1 2604-1102, J10 Conn_01x01, J11 Conn_01x01, J12 Conn_01x01, J13 Conn_01x01, J14 Conn_01x01, J15 Conn_01x01, J16 Conn_01x01, J17 Conn_01x01, J18 Conn_01x01, J19 Conn_01x01, J2 2604-1102, J20 Conn_01x01, J21 Conn_01x01, J22 Conn_01x01, J23 Conn_01x01, J24 Conn_01x01, J25 Conn_01x01, J26 Conn_01x01, J27 Conn_01x01, J28 Conn_01x01, J29 Conn_01x01, J3 Conn_01x01, J30 Conn_01x01, J31 Conn_01x01, J32 Conn_01x01, J33 Conn_01x01, J34 Conn_01x01, J35 Conn_01x01, J4 2604-1102, J5 2604-1102, J6 Conn_01x01, J7 Conn_01x01, J8 Conn_01x01, J9 Conn_01x01, Q1 IPD200N15N3, Q2 IPD200N15N3, Q3 IPD200N15N3, Q4 IPD200N15N3, Q5 IPD200N15N3, U1 ACS730xLCTR-20AB, U10 OPA316, U11 OPA316, U12 OPA316, U13 OPA316, U3 ACS712xLCTR-20A, U4 ACS730xLCTR-20AB, U5 AMC1311, U6 AMC1100DUB, U7 AMC1100DUB, U8 OPA316, U9 OPA316

Commit message: WIP: Layout test V1.1.3
Parts:
- removed JP1, JP10, JP2, JP3, JP4, JP5, JP6, JP7, JP8, JP9: THJP0612AST, Resistor_SMD:R_0612_1632Metric
- added C12: 100nF, Capacitor_SMD:C_1210_3225Metric, F.Cu at (-140.1, 65.5)
- added C12: 100nF, Capacitor_SMD:C_1210_3225Metric, F.Cu at (-178.8, 65.5)
- added C12: 100nF, Capacitor_SMD:C_1210_3225Metric, F.Cu at (-19.1, 49.8)
- added C12: 100nF, Capacitor_SMD:C_1210_3225Metric, F.Cu at (-45.6, 49.8)
- added C12: 100nF, Capacitor_SMD:C_1210_3225Metric, F.Cu at (-71.6, 49.8)
- added C19: 4.7uF, Capacitor_SMD:C_1210_3225Metric, F.Cu at (-128.2, 62.6)
- added C19: 4.7uF, Capacitor_SMD:C_1210_3225Metric, F.Cu at (-167.0, 62.1)
- added C19: 4.7uF, Capacitor_SMD:C_1210_3225Metric, F.Cu at (-6.49, 46.1)
- added C19: 4.7uF, Capacitor_SMD:C_1210_3225Metric, F.Cu at (-33.7, 46.9)
- added C19: 4.7uF, Capacitor_SMD:C_1210_3225Metric, F.Cu at (-59.7, 46.4)
- added C20: 4.7uF, Capacitor_SMD:C_1210_3225Metric, F.Cu at (-136.3, 115.2)
- added C20: 4.7uF, Capacitor_SMD:C_1210_3225Metric, F.Cu at (-55.4, 46.4)
- added C20: 4.7uF, Capacitor_SMD:C_1210_3225Metric, F.Cu at (-174.6, 115.4)
- added C20: 4.7uF, Capacitor_SMD:C_1210_3225Metric, F.Cu at (-123.9, 62.6)
- added C20: 4.7uF, Capacitor_SMD:C_1210_3225Metric, F.Cu at (-162.7, 62.1)
- added C20: 4.7uF, Capacitor_SMD:C_1210_3225Metric, F.Cu at (-13.6, 90.8)
- added C20: 4.7uF, Capacitor_SMD:C_1210_3225Metric, F.Cu at (-40.4, 90.3)
- added C20: 4.7uF, Capacitor_SMD:C_1210_3225Metric, F.Cu at (-66.6, 91.6)
- added C20: 4.7uF, Capacitor_SMD:C_1210_3225Metric, F.Cu at (-2.15, 46.1)
- added C20: 4.7uF, Capacitor_SMD:C_1210_3225Metric, F.Cu at (-29.4, 46.9)
- added C21: 4.7uF, Capacitor_SMD:C_1210_3225Metric, F.Cu at (-128.2, 66.0)
- added C21: 4.7uF, Capacitor_SMD:C_1210_3225Metric, F.Cu at (-167.0, 65.5)
- added C21: 4.7uF, Capacitor_SMD:C_1210_3225Metric, F.Cu at (-6.49, 49.5)
- added C21: 4.7uF, Capacitor_SMD:C_1210_3225Metric, F.Cu at (-33.7, 50.2)
- added C21: 4.7uF, Capacitor_SMD:C_1210_3225Metric, F.Cu at (-59.7, 49.7)
- added C23: 4.7uF, Capacitor_SMD:C_1210_3225Metric, F.Cu at (-171.3, 115.4)
- added C23: 4.7uF, Capacitor_SMD:C_1210_3225Metric, F.Cu at (-55.4, 49.7)
- added C23: 4.7uF, Capacitor_SMD:C_1210_3225Metric, F.Cu at (-123.9, 66.0)
- added C23: 4.7uF, Capacitor_SMD:C_1210_3225Metric, F.Cu at (-133.1, 115.2)
- added C23: 4.7uF, Capacitor_SMD:C_1210_3225Metric, F.Cu at (-162.7, 65.5)
- added C23: 4.7uF, Capacitor_SMD:C_1210_3225Metric, F.Cu at (-13.6, 87.5)
- added C23: 4.7uF, Capacitor_SMD:C_1210_3225Metric, F.Cu at (-40.4, 87.0)
- added C23: 4.7uF, Capacitor_SMD:C_1210_3225Metric, F.Cu at (-66.6, 88.3)
- added C23: 4.7uF, Capacitor_SMD:C_1210_3225Metric, F.Cu at (-2.15, 49.5)
- added C23: 4.7uF, Capacitor_SMD:C_1210_3225Metric, F.Cu at (-29.4, 50.2)
- added C25: 4.7uF, Capacitor_SMD:C_1210_3225Metric, F.Cu at (-128.2, 69.2)
- added C25: 4.7uF, Capacitor_SMD:C_1210_3225Metric, F.Cu at (-167.0, 68.8)
- added C25: 4.7uF, Capacitor_SMD:C_1210_3225Metric, F.Cu at (-6.49, 52.8)
- added C25: 4.7uF, Capacitor_SMD:C_1210_3225Metric, F.Cu at (-33.7, 53.5)
- added C25: 4.7uF, Capacitor_SMD:C_1210_3225Metric, F.Cu at (-59.7, 53.0)
- added C26: 4.7uF, Capacitor_SMD:C_1210_3225Metric, F.Cu at (-168.0, 115.4)
- added C26: 4.7uF, Capacitor_SMD:C_1210_3225Metric, F.Cu at (-55.4, 53.0)
- added C26: 4.7uF, Capacitor_SMD:C_1210_3225Metric, F.Cu at (-129.8, 115.2)
- added C26: 4.7uF, Capacitor_SMD:C_1210_3225Metric, F.Cu at (-123.9, 69.2)
- added C26: 4.7uF, Capacitor_SMD:C_1210_3225Metric, F.Cu at (-162.7, 68.8)
- added C26: 4.7uF, Capacitor_SMD:C_1210_3225Metric, F.Cu at (-13.6, 84.2)
- added C26: 4.7uF, Capacitor_SMD:C_1210_3225Metric, F.Cu at (-40.4, 83.8)
- added C26: 4.7uF, Capacitor_SMD:C_1210_3225Metric, F.Cu at (-66.6, 85.0)
- added C26: 4.7uF, Capacitor_SMD:C_1210_3225Metric, F.Cu at (-2.15, 52.8)
- added C26: 4.7uF, Capacitor_SMD:C_1210_3225Metric, F.Cu at (-29.4, 53.5)
- added C39: 100nF, Capacitor_SMD:C_1210_3225Metric, F.Cu at (-140.1, 62.2)
- added C39: 100nF, Capacitor_SMD:C_1210_3225Metric, F.Cu at (-178.8, 62.2)
- added C39: 100nF, Capacitor_SMD:C_1210_3225Metric, F.Cu at (-19.1, 46.5)
- added C39: 100nF, Capacitor_SMD:C_1210_3225Metric, F.Cu at (-45.6, 46.5)
- added C39: 100nF, Capacitor_SMD:C_1210_3225Metric, F.Cu at (-71.6, 46.5)
- added C39: 100nF, Capacitor_SMD:C_1210_3225Metric, F.Cu at (64.0, 51.4)
- added C40: 100nF, Capacitor_SMD:C_1210_3225Metric, F.Cu at (111.5, 51.6)
- added C41: 100nF, Capacitor_SMD:C_1210_3225Metric, F.Cu at (-140.1, 68.8)
- added C41: 100nF, Capacitor_SMD:C_1210_3225Metric, F.Cu at (-178.8, 68.8)
- added C41: 100nF, Capacitor_SMD:C_1210_3225Metric, F.Cu at (-19.1, 53.0)
- added C41: 100nF, Capacitor_SMD:C_1210_3225Metric, F.Cu at (-45.6, 53.0)
- added C41: 100nF, Capacitor_SMD:C_1210_3225Metric, F.Cu at (-71.6, 53.0)
- added C41: 100nF, Capacitor_SMD:C_1210_3225Metric, F.Cu at (57.5, 51.4)
- added C42: 100nF, Capacitor_SMD:C_1210_3225Metric, F.Cu at (118.0, 51.6)
- added Cs4: C_Small, Capacitor_SMD:C_0805_2012Metric, F.Cu at (-136.6, 87.5)
- added Cs4: C_Small, Capacitor_SMD:C_0805_2012Metric, F.Cu at (-175.4, 87.5)
- added Cs4: C_Small, Capacitor_SMD:C_0805_2012Metric, F.Cu at (-15.6, 71.8)
- added Cs4: C_Small, Capacitor_SMD:C_0805_2012Metric, F.Cu at (-42.1, 71.8)
- added Cs4: C_Small, Capacitor_SMD:C_0805_2012Metric, F.Cu at (-68.1, 71.8)
- added D4: STPS0520Z, Diode_SMD:D_SOD-123, F.Cu at (-142.0, 73.5)
- added D4: STPS0520Z, Diode_SMD:D_SOD-123, F.Cu at (-180.7, 73.5)
- added D4: STPS0520Z, Diode_SMD:D_SOD-123, F.Cu at (-21.0, 57.8)
- added D4: STPS0520Z, Diode_SMD:D_SOD-123, F.Cu at (-47.5, 57.8)
- added D4: STPS0520Z, Diode_SMD:D_SOD-123, F.Cu at (-73.5, 57.8)
- added D5: STPS0520Z, Diode_SMD:D_SOD-123, F.Cu at (-142.0, 79.0)
- added D5: STPS0520Z, Diode_SMD:D_SOD-123, F.Cu at (-180.7, 79.0)
- added D5: STPS0520Z, Diode_SMD:D_SOD-123, F.Cu at (-21.0, 63.3)
- added D5: STPS0520Z, Diode_SMD:D_SOD-123, F.Cu at (-47.5, 63.3)
- added D5: STPS0520Z, Diode_SMD:D_SOD-123, F.Cu at (-73.5, 63.3)
- added D_L2: STTH1002CB, Diode_SMD:D_SOD-123, F.Cu at (-134.4, 85.0)
- added D_L2: STTH1002CB, Diode_SMD:D_SOD-123, F.Cu at (-173.2, 85.0)
- added D_L2: STTH1002CB, Diode_SMD:D_SOD-123, F.Cu at (-13.4, 69.2)
- added D_L2: STTH1002CB, Diode_SMD:D_SOD-123, F.Cu at (-39.9, 69.2)
- added D_L2: STTH1002CB, Diode_SMD:D_SOD-123, F.Cu at (-65.9, 69.2)
- added F2: Nano2 fuse holder, Footprints:Fuse_holder_omni_blok, F.Cu at (-110.5, 144.3)
- added F2: Nano2 fuse holder, Footprints:Fuse_holder_omni_blok, F.Cu at (-188.7, 133.2)
- added F2: Nano2 fuse holder, Footprints:Fuse_holder_omni_blok, F.Cu at (-173.8, 133.5)
- added F2: Nano2 fuse holder, Footprints:Fuse_holder_omni_blok, F.Cu at (-90.8, 117.0)
- added F2: Nano2 fuse holder, Footprints:Fuse_holder_omni_blok, F.Cu at (-52.4, 115.5)
- added F2: Nano2 fuse holder, Footprints:Fuse_holder_omni_blok, F.Cu at (-30.9, 115.5)
- added F2: Nano2 fuse holder, Footprints:Fuse_holder_omni_blok, F.Cu at (-9.94, 115.8)
- added HS1: Heatsink_Pad, Footprints:custom_heatsink, F.Cu at (199.8, 3.75)
- added J1: 2604-1102, Footprints:WAGO-2604-1102, F.Cu at (-123.8, 140.0)
- added J1: 2604-1102, Footprints:WAGO-2604-1102, F.Cu at (-53.8, 122.8)
- added J1: 2604-1102, Footprints:WAGO-2604-1102, F.Cu at (-34.2, 122.8)
- added J1: 2604-1102, Footprints:WAGO-2604-1102, F.Cu at (-24.5, 122.8)
- added J1: 2604-1102, Footprints:WAGO-2604-1102, F.Cu at (-180.2, 139.8)
- added J1: 2604-1102, Footprints:WAGO-2604-1102, F.Cu at (-190.2, 139.8)
- added J1: 2604-1102, Footprints:WAGO-2604-1102, F.Cu at (-137.5, 140.0)
- added J1: 2604-1102, Footprints:WAGO-2604-1102, F.Cu at (-160.5, 139.8)
- added J1: 2604-1102, Footprints:WAGO-2604-1102, F.Cu at (-11.8, 122.8)
- added J1: 2604-1102, Footprints:WAGO-2604-1102, F.Cu at (-95.0, 123.0)
- added J1: 2604-1102, Footprints:WAGO-2604-1102, F.Cu at (-104.8, 123.0)
- added J1: 2604-1102, Footprints:WAGO-2604-1102, F.Cu at (-43.8, 122.8)
- added J21: Conn_01x01, Footprints:0906_millmax, B.Cu at (-144.2, 72.0)
- added J21: Conn_01x01, Footprints:0906_millmax, B.Cu at (-183.2, 72.0)
- added J21: Conn_01x01, Footprints:0906_millmax, B.Cu at (-23.4, 56.3)
- added J21: Conn_01x01, Footprints:0906_millmax, B.Cu at (-49.7, 56.3)
- added J21: Conn_01x01, Footprints:0906_millmax, B.Cu at (-76.0, 56.3)
- added J22: Conn_01x01, Footprints:0906_millmax, B.Cu at (-144.2, 74.6)
- added J22: Conn_01x01, Footprints:0906_millmax, B.Cu at (-183.2, 74.6)
- added J22: Conn_01x01, Footprints:0906_millmax, B.Cu at (-23.4, 58.8)
- added J22: Conn_01x01, Footprints:0906_millmax, B.Cu at (-49.7, 58.8)
- added J22: Conn_01x01, Footprints:0906_millmax, B.Cu at (-76.0, 58.8)
- added J23: Conn_01x01, Footprints:0906_millmax, B.Cu at (-144.2, 80.6)
- added J23: Conn_01x01, Footprints:0906_millmax, B.Cu at (-182.9, 80.6)
- added J23: Conn_01x01, Footprints:0906_millmax, B.Cu at (-23.2, 64.8)
- added J23: Conn_01x01, Footprints:0906_millmax, B.Cu at (-49.7, 64.8)
- added J23: Conn_01x01, Footprints:0906_millmax, B.Cu at (-75.7, 64.8)
- added J24: Conn_01x01, Footprints:0906_millmax, B.Cu at (-144.2, 83.1)
- added J24: Conn_01x01, Footprints:0906_millmax, B.Cu at (-182.9, 83.1)
- added J24: Conn_01x01, Footprints:0906_millmax, B.Cu at (-23.2, 67.4)
- added J24: Conn_01x01, Footprints:0906_millmax, B.Cu at (-49.7, 67.4)
- added J24: Conn_01x01, Footprints:0906_millmax, B.Cu at (-75.7, 67.4)
- added J36: 2604-1102, Footprints:WAGO-2604-1102, F.Cu at (69.7, 127.0)
- added L1: 47uH, Footprints:WE-HCF-2013, F.Cu at (-174.2, 100.5)
- added L1: 47uH, Footprints:WE-HCF-2013, F.Cu at (-135.5, 100.5)
- added Q4: IPD200N15N3, Package_TO_SOT_SMD:TO-252-2, F.Cu at (-145.5, 142.3)
- added Q4: IPD200N15N3, Package_TO_SOT_SMD:TO-252-2, F.Cu at (-134.1, 68.9)
- added Q4: IPD200N15N3, Package_TO_SOT_SMD:TO-252-2, F.Cu at (-172.8, 68.9)
- added Q4: IPD200N15N3, Package_TO_SOT_SMD:TO-252-2, F.Cu at (-63.0, 125.4)
- added Q4: IPD200N15N3, Package_TO_SOT_SMD:TO-252-2, F.Cu at (-13.1, 53.1)
- added Q4: IPD200N15N3, Package_TO_SOT_SMD:TO-252-2, F.Cu at (-39.6, 53.1)
- added Q4: IPD200N15N3, Package_TO_SOT_SMD:TO-252-2, F.Cu at (-65.6, 53.1)
- added Q5: IPD200N15N3, Package_TO_SOT_SMD:TO-252-2, F.Cu at (-132.4, 80.2)
- added Q5: IPD200N15N3, Package_TO_SOT_SMD:TO-252-2, F.Cu at (-171.2, 80.2)
- added Q5: IPD200N15N3, Package_TO_SOT_SMD:TO-252-2, F.Cu at (-11.4, 64.4)
- added Q5: IPD200N15N3, Package_TO_SOT_SMD:TO-252-2, F.Cu at (-37.9, 64.4)
- added Q5: IPD200N15N3, Package_TO_SOT_SMD:TO-252-2, F.Cu at (-63.9, 64.4)
- added R33: 0, Resistor_SMD:R_0805_2012Metric, F.Cu at (-139.4, 72.4)
- added R33: 0, Resistor_SMD:R_0805_2012Metric, F.Cu at (-178.1, 72.4)
- added R33: 0, Resistor_SMD:R_0805_2012Metric, F.Cu at (-18.4, 56.6)
- added R33: 0, Resistor_SMD:R_0805_2012Metric, F.Cu at (-44.9, 56.6)
- added R33: 0, Resistor_SMD:R_0805_2012Metric, F.Cu at (-70.9, 56.6)
- added R34: 0, Resistor_SMD:R_0805_2012Metric, F.Cu at (-139.4, 77.9)
- added R34: 0, Resistor_SMD:R_0805_2012Metric, F.Cu at (-178.1, 77.9)
- added R34: 0, Resistor_SMD:R_0805_2012Metric, F.Cu at (-18.4, 62.1)
- added R34: 0, Resistor_SMD:R_0805_2012Metric, F.Cu at (-44.9, 62.1)
- added R34: 0, Resistor_SMD:R_0805_2012Metric, F.Cu at (-70.9, 62.1)
- added R35: 1k, Resistor_SMD:R_0805_2012Metric, F.Cu at (-134.5, 73.8)
- added R35: 1k, Resistor_SMD:R_0805_2012Metric, F.Cu at (-173.2, 73.8)
- added R35: 1k, Resistor_SMD:R_0805_2012Metric, F.Cu at (-13.5, 58.1)
- added R35: 1k, Resistor_SMD:R_0805_2012Metric, F.Cu at (-40.0, 58.1)
- added R35: 1k, Resistor_SMD:R_0805_2012Metric, F.Cu at (-66.0, 58.1)
- added R36: 1k, Resistor_SMD:R_0805_2012Metric, F.Cu at (-137.0, 81.0)
- added R36: 1k, Resistor_SMD:R_0805_2012Metric, F.Cu at (-175.7, 81.0)
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Connections:
- J1 pad 3: Net-(F3-Pad2) -> Net-(F2-Pad2)
- J1 pad 4: Net-(F3-Pad2) -> Net-(F2-Pad2)
Routing:
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- added copper zone on B.Cu, net (none)
- added copper zone on F.Cu, net (none)
- added copper zone on In2.Cu, net /N
- added copper zone on B.Cu, net /SW_Node1
- added copper zone on B.Cu, net /SW_Node2
- added copper zone on In2.Cu, net Net-(F2-Pad2)
- added copper zone on B.Cu, net Net-(HS1-Pad1)
- removed copper zone on In1.Cu, net /SW_Node1
- removed copper zone on In1.Cu, net /SW_Node2
- removed copper zone on B.Cu, net /VI_LOW1
- removed copper zone on B.Cu, net /VI_LOW2
- removed copper zone on In1.Cu, net /V_Out
- removed copper zone on B.Cu, net GNDREF
- removed copper zone on In2.Cu, net GNDREF
- removed copper zone on B.Cu, net Net-(F1-Pad2)
- removed copper zone on B.Cu, net Net-(L1-Pad1)
- removed copper zone on B.Cu, net Net-(L2-Pad1)

Commit message: Added the third power leg. Changed the unductor to 33uH SRP1510. Started a draft of power layout
Parts:
- removed the C12 at (-140.1, 65.5)
- removed the C12 at (-178.8, 65.5)
- removed the C12 at (-19.1, 49.8)
- removed the C12 at (-45.6, 49.8)
- removed the C12 at (-71.6, 49.8)
- removed the C12 at (60.8, 51.4)
- removed the C19 at (-128.2, 62.6)
- removed the C19 at (-167.0, 62.1)
- removed the C19 at (-6.49, 46.1)
- removed the C19 at (-33.7, 46.9)
- removed the C19 at (-59.7, 46.4)
- removed the C19 at (68.7, 55.7)
- removed the C20 at (-136.3, 115.2)
- removed the C20 at (-55.4, 46.4)
- removed the C20 at (68.7, 51.4)
- removed the C20 at (-174.6, 115.4)
- removed the C20 at (-123.9, 62.6)
- removed the C20 at (-162.7, 62.1)
- removed the C20 at (-13.6, 90.8)
- removed the C20 at (-40.4, 90.3)
- removed the C20 at (-66.6, 91.6)
- removed the C20 at (-2.15, 46.1)
- removed the C20 at (-29.4, 46.9)
- removed the C21 at (-128.2, 66.0)
- removed the C21 at (-167.0, 65.5)
- removed the C21 at (-6.49, 49.5)
- removed the C21 at (-33.7, 50.2)
- removed the C21 at (-59.7, 49.7)
- removed the C21 at (72.0, 55.7)
- removed the C23 at (-171.3, 115.4)
- removed the C23 at (-55.4, 49.7)
- removed the C23 at (72.0, 51.4)
- removed the C23 at (-123.9, 66.0)
- removed the C23 at (-133.1, 115.2)
- removed the C23 at (-162.7, 65.5)
- removed the C23 at (-13.6, 87.5)
- removed the C23 at (-40.4, 87.0)
- removed the C23 at (-66.6, 88.3)
- removed the C23 at (-2.15, 49.5)
- removed the C23 at (-29.4, 50.2)
- removed the C25 at (-128.2, 69.2)
- removed the C25 at (-167.0, 68.8)
- removed the C25 at (-6.49, 52.8)
- removed the C25 at (-33.7, 53.5)
- removed the C25 at (-59.7, 53.0)
- removed the C25 at (75.2, 55.7)
- removed the C26 at (-168.0, 115.4)
- removed the C26 at (-55.4, 53.0)
- removed the C26 at (75.2, 51.4)
- removed the C26 at (-129.8, 115.2)
- removed the C26 at (-123.9, 69.2)
- removed the C26 at (-162.7, 68.8)
- removed the C26 at (-13.6, 84.2)
- removed the C26 at (-40.4, 83.8)
- removed the C26 at (-66.6, 85.0)
- removed the C26 at (-2.15, 52.8)
- removed the C26 at (-29.4, 53.5)
- removed the C39 at (-140.1, 62.2)
- removed the C39 at (-178.8, 62.2)
- removed the C39 at (-19.1, 46.5)
- removed the C39 at (-45.6, 46.5)
- removed the C39 at (-71.6, 46.5)
- removed the C39 at (64.0, 51.4)
- removed the C41 at (-140.1, 68.8)
- removed the C41 at (-178.8, 68.8)
- removed the C41 at (-19.1, 53.0)
- removed the C41 at (-45.6, 53.0)
- removed the C41 at (-71.6, 53.0)
- removed the C41 at (57.5, 51.4)
- removed Cs3: C_Small, Capacitor_SMD:C_0805_2012Metric
- removed the Cs4 at (-136.6, 87.5)
- removed the Cs4 at (-175.4, 87.5)
- removed the Cs4 at (-15.6, 71.8)
- removed the Cs4 at (-42.1, 71.8)
- removed the Cs4 at (-68.1, 71.8)
- removed the Cs4 at (68.5, 75.1)
- removed the D4 at (-142.0, 73.5)
- removed the D4 at (-180.7, 73.5)
- removed the D4 at (-21.0, 57.8)
- removed the D4 at (-47.5, 57.8)
- removed the D4 at (-73.5, 57.8)
- removed the D4 at (52.5, 64.3)
- removed the D5 at (-142.0, 79.0)
- removed the D5 at (-180.7, 79.0)
- removed the D5 at (-21.0, 63.3)
- removed the D5 at (-47.5, 63.3)
- removed the D5 at (-73.5, 63.3)
- removed the D5 at (53.0, 77.3)
- removed D_H1, D_H2: STTH1002CB, Diode_SMD:D_SOD-123
- removed the D_L2 at (-134.4, 85.0)
- removed the D_L2 at (-173.2, 85.0)
- removed the D_L2 at (-13.4, 69.2)
- removed the D_L2 at (-39.9, 69.2)
- removed the D_L2 at (-65.9, 69.2)
- removed the D_L2 at (66.0, 72.9)
- removed the F2 at (-110.5, 144.3)
- removed the F2 at (-188.7, 133.2)
- removed the F2 at (-173.8, 133.5)
- removed the F2 at (-90.8, 117.0)
- removed the F2 at (-52.4, 115.5)
- removed the F2 at (-30.9, 115.5)
- removed the F2 at (-9.94, 115.8)
- removed the F2 at (47.4, 132.8)
- removed the J1 at (-123.8, 140.0)
- removed the J1 at (-53.8, 122.8)
- removed the J1 at (-34.2, 122.8)
- removed the J1 at (-24.5, 122.8)
- removed the J1 at (59.5, 127.0)
- removed the J1 at (-180.2, 139.8)
- removed the J1 at (-190.2, 139.8)
- removed the J1 at (-137.5, 140.0)
- removed the J1 at (-160.5, 139.8)
- removed the J1 at (-11.8, 122.8)
- removed the J1 at (-95.0, 123.0)
- removed the J1 at (-104.8, 123.0)
- removed the J1 at (-43.8, 122.8)
- removed the J21 at (-144.2, 72.0)
- removed the J21 at (-183.2, 72.0)
- removed the J21 at (-23.4, 56.3)
- removed the J21 at (-49.7, 56.3)
- removed the J21 at (-76.0, 56.3)
- removed the J21 at (50.8, 66.0)
- removed the J22 at (-144.2, 74.6)
- removed the J22 at (-183.2, 74.6)
- removed the J22 at (-23.4, 58.8)
- removed the J22 at (-49.7, 58.8)
- removed the J22 at (-76.0, 58.8)
- removed the J22 at (50.8, 68.6)
- removed the J23 at (-144.2, 80.6)
- removed the J23 at (-182.9, 80.6)
- removed the J23 at (-23.2, 64.8)
- removed the J23 at (-49.7, 64.8)
- removed the J23 at (-75.7, 64.8)
- removed the J23 at (50.8, 78.8)
- removed the J24 at (-144.2, 83.1)
- removed the J24 at (-182.9, 83.1)
- removed the J24 at (-23.2, 67.4)
- removed the J24 at (-49.7, 67.4)
- removed the J24 at (-75.7, 67.4)
- removed the J24 at (50.8, 81.4)
- removed the L1 at (-174.2, 100.5)
- removed the L1 at (-135.5, 100.5)
- removed the L1 at (92.0, 58.0)
- removed the Q4 at (-145.5, 142.3)
- removed the Q4 at (-134.1, 68.9)
- removed the Q4 at (-172.8, 68.9)
- removed the Q4 at (-63.0, 125.4)
- removed the Q4 at (-13.1, 53.1)
- removed the Q4 at (-39.6, 53.1)
- removed the Q4 at (-65.6, 53.1)
- removed the Q4 at (60.4, 59.6)
- removed the Q5 at (-132.4, 80.2)
- removed the Q5 at (-171.2, 80.2)
- removed the Q5 at (-11.4, 64.4)
- removed the Q5 at (-37.9, 64.4)
- removed the Q5 at (-63.9, 64.4)
- removed the Q5 at (60.4, 72.2)
- removed the R33 at (-139.4, 72.4)
- removed the R33 at (-178.1, 72.4)
- removed the R33 at (-18.4, 56.6)
- removed the R33 at (-44.9, 56.6)
- removed the R33 at (-70.9, 56.6)
- removed the R33 at (55.1, 63.1)
- removed the R34 at (-139.4, 77.9)
- removed the R34 at (-178.1, 77.9)
- removed the R34 at (-18.4, 62.1)
- removed the R34 at (-44.9, 62.1)
- removed the R34 at (-70.9, 62.1)
- removed the R34 at (55.6, 76.1)
- removed the R35 at (-134.5, 73.8)
- removed the R35 at (-173.2, 73.8)
- removed the R35 at (-13.5, 58.1)
- removed the R35 at (-40.0, 58.1)
- removed the R35 at (-66.0, 58.1)
- removed the R35 at (60.0, 64.6)
- removed the R36 at (-137.0, 81.0)
- removed the R36 at (-175.7, 81.0)
- removed the R36 at (-16.0, 65.2)
- removed the R36 at (-42.5, 65.2)
- removed the R36 at (-68.5, 65.2)
- removed the R36 at (58.0, 79.2)
- removed the R5 at (-139.4, 74.4)
- removed the R5 at (-178.1, 74.4)
- removed the R5 at (-18.4, 58.6)
- removed the R5 at (-44.9, 58.6)
- removed the R5 at (-70.9, 58.6)
- removed the R5 at (55.1, 65.1)
- removed the R6 at (-139.4, 79.9)
- removed the R6 at (-178.1, 79.9)
- removed the R6 at (-18.4, 64.1)
- removed the R6 at (-44.9, 64.1)
- removed the R6 at (-70.9, 64.1)
- removed the R6 at (55.6, 78.1)
- removed REF** (x3): L_Vishay_IHLP-6767, Inductor_SMD:L_Vishay_IHLP-6767
- removed Rs3: R_Small, Resistor_SMD:R_0805_2012Metric
- removed the Rs4 at (-133.2, 87.5)
- removed the Rs4 at (-172.0, 87.5)
- removed the Rs4 at (-12.2, 71.7)
- removed the Rs4 at (-38.7, 71.7)
- removed the Rs4 at (-64.7, 71.7)
- removed the Rs4 at (68.5, 71.7)
- removed the U1 at (-128.0, 121.5)
- removed the U1 at (-162.8, 119.5)
- removed the U1 at (-88.8, 102.8)
- removed the U1 at (-60.0, 94.8)
- removed the U1 at (-34.2, 94.8)
- removed the U1 at (-8.00, 95.0)
- removed the U1 at (75.5, 95.0)
- removed the U3 at (-118.2, 121.5)
- removed the U3 at (115.0, 105.0)
- removed the U5 at (-91.5, 109.5)
- removed the U5 at (-120.2, 131.0)
- removed the U5 at (113.0, 114.5)
- removed the U7 at (-182.8, 121.5)
- removed the U7 at (-143.2, 122.0)
- removed the U7 at (1.50, 105.8)
- removed the U7 at (-49.8, 106.0)
- removed the U7 at (-34.8, 105.0)
- removed the U7 at (68.5, 114.6)
- added C12: 100nF, Capacitor_SMD:C_1210_3225Metric, F.Cu at (107.8, 87.1)
- added C19: 4.7uF, Capacitor_SMD:C_1210_3225Metric, F.Cu at (-34.3, 21.6)
- added C20: 4.7uF, Capacitor_SMD:C_1210_3225Metric, F.Cu at (-21.2, 5.06)
- added C21: 4.7uF, Capacitor_SMD:C_1210_3225Metric, F.Cu at (-18.0, -1.14)
- added C23: 4.7uF, Capacitor_SMD:C_1210_3225Metric, F.Cu at (-70.2, 57.1)
- added C25: 4.7uF, Capacitor_SMD:C_1210_3225Metric, F.Cu at (-56.5, 42.5)
- added C26: 4.7uF, Capacitor_SMD:C_1210_3225Metric, F.Cu at (-50.8, 38.2)
- added C39: 100nF, Capacitor_SMD:C_1210_3225Metric, F.Cu at (107.8, 90.3)
- added C41: 100nF, Capacitor_SMD:C_1210_3225Metric, F.Cu at (107.8, 93.6)
- added C43: 4.7uF, Capacitor_SMD:C_1210_3225Metric, F.Cu at (-58.1, 106.3)
- added C44: 4.7uF, Capacitor_SMD:C_1210_3225Metric, F.Cu at (-43.5, 88.8)
- added C45: 4.7uF, Capacitor_SMD:C_1210_3225Metric, F.Cu at (-37.7, 85.4)
- added C46: 1nF, Capacitor_SMD:C_0805_2012Metric, F.Cu at (-23.5, 76.8)
- added C47: 100nF, Capacitor_SMD:C_0805_2012Metric, F.Cu at (-53.0, 105.7)
- added C48: 100nF, Capacitor_SMD:C_1210_3225Metric, F.Cu at (107.4, 125.4)
- added C49: 100nF, Capacitor_SMD:C_1210_3225Metric, F.Cu at (107.4, 122.1)
- added C50: 100nF, Capacitor_SMD:C_1210_3225Metric, F.Cu at (107.3, 118.6)
- added C51: 100nF, Capacitor_SMD:C_0805_2012Metric, F.Cu at (-48.0, 101.0)
- added C52: 100nF, Capacitor_SMD:C_0805_2012Metric, F.Cu at (-58.7, 109.9)
- added C53: 100nF, Capacitor_SMD:C_0805_2012Metric, F.Cu at (-42.2, 96.7)
- added C54: 100nF, Capacitor_SMD:C_0805_2012Metric, F.Cu at (-38.4, 93.3)
- added Cs4: C_Small, Capacitor_SMD:C_0805_2012Metric, F.Cu at (-45.8, 37.8)
- added D1: STPS0520Z, Diode_SMD:D_SOD-123, F.Cu at (-69.7, 99.9)
- added D4: STPS0520Z, Diode_SMD:D_SOD-123, F.Cu at (101.4, 91.1)
- added D5: STPS0520Z, Diode_SMD:D_SOD-123, F.Cu at (95.3, 91.0)
- added D6: STPS0520Z, Diode_SMD:D_SOD-123, F.Cu at (-47.4, 97.8)
- added D_L2: STTH1002CB, Diode_SMD:D_SOD-123, F.Cu at (-45.6, 19.3)
- added D_L3: STTH1002CB, Diode_SMD:D_SOD-123, F.Cu at (-43.4, 85.0)
- added F2: Nano2 fuse holder, Footprints:Fuse_holder_omni_blok, F.Cu at (-26.6, -0.17)
- added F5: Nano2 fuse holder, Footprints:Fuse_holder_omni_blok, F.Cu at (-66.7, 107.3)
- added J1: 2604-1102, Footprints:WAGO-2604-1102, F.Cu at (-71.2, 0.47)
- added J21: Conn_01x01, Footprints:0906_millmax, F.Cu at (-23.1, 34.0)
- added J22: Conn_01x01, Footprints:0906_millmax, F.Cu at (-37.0, 48.1)
- added J23: Conn_01x01, Footprints:0906_millmax, F.Cu at (-80.7, 58.6)
- added J24: Conn_01x01, Footprints:0906_millmax, F.Cu at (-11.5, 19.3)
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Connections:
- Cs1 pad 2: /SW_Node1 -> GNDREF
- Rs1 pad 1: /V_Out -> /SW_Node3
- U5 pad 1: (no net) -> +5P
- U5 pad 2: (no net) -> /VIHigh+
- U5 pad 3: (no net) -> GNDREF
- U5 pad 4: (no net) -> GNDREF
- U5 pad 5: (no net) -> /DGND
- U5 pad 6: (no net) -> Net-(R8-Pad1)
- U5 pad 7: (no net) -> Net-(R7-Pad1)
- U5 pad 8: (no net) -> +5VD
Routing:
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- removed copper zone on B.Cu, net (none)
- removed copper zone on F.Cu, net (none)
- removed copper zone on In2.Cu, net +5V
- removed copper zone on In2.Cu, net +5VD
- removed copper zone on B.Cu, net /DGND
- removed copper zone on In1.Cu, net /DGND
- removed copper zone on B.Cu, net /N
- removed copper zone on F.Cu, net /N
- removed copper zone on In1.Cu, net /N
- removed copper zone on In2.Cu, net /N
- removed copper zone on B.Cu, net /SW_Node1
- removed copper zone on F.Cu, net /SW_Node1
- removed copper zone on B.Cu, net /SW_Node2
- removed copper zone on F.Cu, net /SW_Node2
- removed copper zone on F.Cu, net /VI_High
- removed copper zone on F.Cu, net /VI_LOW1
- removed copper zone on In2.Cu, net /VI_LOW1
- removed copper zone on F.Cu, net /VI_LOW2
- removed copper zone on In2.Cu, net /VI_LOW2
- removed copper zone on B.Cu, net /V_Out
- removed copper zone on F.Cu, net /V_Out
- removed copper zone on In2.Cu, net /V_Out
- removed copper zone on F.Cu, net GNDREF
- removed copper zone on In1.Cu, net GNDREF
- removed copper zone on F.Cu, net Net-(C13-Pad2)
- removed copper zone on F.Cu, net Net-(F1-Pad2)
- removed copper zone on In2.Cu, net Net-(F1-Pad2)
- removed copper zone on F.Cu, net Net-(F2-Pad2)
- removed copper zone on In2.Cu, net Net-(F2-Pad2)
- removed copper zone on F.Cu, net Net-(F3-Pad2)
- removed copper zone on B.Cu, net Net-(HS1-Pad1)
- removed copper zone on F.Cu, net Net-(HS1-Pad1)
- removed copper zone on In1.Cu, net Net-(HS1-Pad1)
- removed copper zone on F.Cu, net Net-(L1-Pad1)
- removed copper zone on In2.Cu, net Net-(L1-Pad1)
- removed copper zone on F.Cu, net Net-(L2-Pad1)
- removed copper zone on F.Cu, net Net-(Q1-Pad1)
- removed copper zone on F.Cu, net Net-(Q2-Pad1)
- removed copper zone on F.Cu, net Net-(Q4-Pad1)
- removed copper zone on F.Cu, net Net-(Q5-Pad1)

Commit message: First attempt at creating a complete layout.
Parts:
- J10, J13, J16, J19, J21, J22, J23, J24: moved to B.Cu
- moved J36 222.0 mm to (125.7, 129.2)
- moved C28 219.4 mm to (112.7, 103.5), turned to 180 degrees
- moved U6 214.8 mm to (118.1, 109.5)
- moved C24 214.4 mm to (113.0, 93.5), turned to 180 degrees
- moved C22 209.0 mm to (112.2, 96.9), turned to 90 degrees
- moved C31 207.5 mm to (120.1, 94.0), turned to 90 degrees
- moved F3 203.4 mm to (119.0, 134.3), turned to 270 degrees
- moved J10 187.0 mm to (132.8, 109.6), turned to 90 degrees
- moved U9 181.6 mm to (129.2, 109.0)
- moved R28 180.4 mm to (119.1, 99.6)
- moved C34 178.7 mm to (130.2, 105.6), turned to 90 degrees
- moved R10 177.8 mm to (126.0, 110.6)
- moved R9 177.5 mm to (126.0, 108.3)
- moved R17 177.0 mm to (129.3, 111.3)
- moved J13 176.3 mm to (132.8, 107.1), turned to 90 degrees
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Routing:
- net /SW_Node2: track 0.00 -> 31.5 mm, vias 0 -> 10
- net GNDREF: track 0.00 -> 19.8 mm, vias 0 -> 12
- net /DGND: track 0.00 -> 15.2 mm, vias 0 -> 10
- net +5VD: track 0.00 -> 13.6 mm, vias 0 -> 4
- net /VI_LOW2: track 0.00 -> 11.8 mm, vias 0 -> 6
- net /N: track 0.00 -> 8.06 mm, vias 0 -> 9
- net Net-(Q4-Pad1): track 0.00 -> 7.05 mm
- net Net-(Q5-Pad1): track 0.00 -> 7.04 mm
- net /IILow2: track 0.00 -> 5.18 mm
- net /PWM_H2: track 0.00 -> 5.10 mm
- net /PWM_L2: track 0.00 -> 4.94 mm
- net /VILow2+: track 0.00 -> 4.61 mm
- net /IILow2_op: track 0.00 -> 4.42 mm
- net /VILow2_op: track 0.00 -> 4.10 mm
- net Net-(R23-Pad2): track 0.00 -> 3.89 mm
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- added copper zone on B.Cu, net (none)
- added copper zone on In2.Cu, net +5VD
- added copper zone on F.Cu, net /DGND
- added copper zone on In1.Cu, net /DGND
- added copper zone on F.Cu, net /N
- added copper zone on In1.Cu, net /N
- added copper zone on F.Cu, net /SW_Node2
- added copper zone on F.Cu, net /VI_LOW2
- added copper zone on F.Cu, net /V_Out
- added copper zone on F.Cu, net GNDREF
- added copper zone on In1.Cu, net GNDREF
- added copper zone on In2.Cu, net GNDREF
- added copper zone on F.Cu, net Net-(L2-Pad1)

Commit message: Rearranged the schematic for a 3 leg version using subsheets.
Parts:
- removed the J3 at (-12.9, 23.2)
- removed the J34 at (-45.7, 49.6)
- added C10: 4.7uF, Capacitor_SMD:C_1210_3225Metric, F.Cu at (98.2, 111.9)
- added C10: 4.7uF, Capacitor_SMD:C_1210_3225Metric, F.Cu at (98.1, 87.5)
- added C10: 4.7uF, Capacitor_SMD:C_1210_3225Metric, F.Cu at (98.2, 63.2)
- added C12: 100nF, Capacitor_SMD:C_0805_2012Metric, F.Cu at (55.8, 56.2)
- added C21: 4.7uF, Capacitor_SMD:C_1210_3225Metric, F.Cu at (52.9, 93.0)
- added C21: 4.7uF, Capacitor_SMD:C_1210_3225Metric, F.Cu at (52.9, 68.5)
- added C21: 4.7uF, Capacitor_SMD:C_1210_3225Metric, F.Cu at (52.9, 86.7)
- added C22: 1nF, Capacitor_SMD:C_0805_2012Metric, F.Cu at (112.2, 110.1)
- added C22: 1nF, Capacitor_SMD:C_0805_2012Metric, F.Cu at (112.3, 86.1)
- added C22: 1nF, Capacitor_SMD:C_0805_2012Metric, F.Cu at (112.4, 61.7)
- added C23: 4.7uF, Capacitor_SMD:C_1210_3225Metric, F.Cu at (57.7, 93.1)
- added C23: 4.7uF, Capacitor_SMD:C_1210_3225Metric, F.Cu at (57.7, 68.6)
- added C23: 4.7uF, Capacitor_SMD:C_1210_3225Metric, F.Cu at (57.7, 86.8)
- added C24: 100nF, Capacitor_SMD:C_0805_2012Metric, F.Cu at (113.0, 106.7)
- added C24: 100nF, Capacitor_SMD:C_0805_2012Metric, F.Cu at (113.2, 82.7)
- added C24: 100nF, Capacitor_SMD:C_0805_2012Metric, F.Cu at (113.2, 58.3)
- added C25: 4.7uF, Capacitor_SMD:C_1210_3225Metric, F.Cu at (52.9, 89.9)
- added C25: 4.7uF, Capacitor_SMD:C_1210_3225Metric, F.Cu at (52.9, 65.4)
- added C25: 4.7uF, Capacitor_SMD:C_1210_3225Metric, F.Cu at (52.9, 62.3)
- added C26: 4.7uF, Capacitor_SMD:C_1210_3225Metric, F.Cu at (57.7, 89.9)
- added C26: 4.7uF, Capacitor_SMD:C_1210_3225Metric, F.Cu at (57.7, 65.4)
- added C26: 4.7uF, Capacitor_SMD:C_1210_3225Metric, F.Cu at (57.7, 62.3)
- added C28: 100nF, Capacitor_SMD:C_0805_2012Metric, F.Cu at (106.2, 92.5)
- added C28: 100nF, Capacitor_SMD:C_0805_2012Metric, F.Cu at (106.2, 68.0)
- added C28: 100nF, Capacitor_SMD:C_0805_2012Metric, F.Cu at (106.3, 43.6)
- added C31: 100nF, Capacitor_SMD:C_0805_2012Metric, F.Cu at (120.1, 107.2)
- added C31: 100nF, Capacitor_SMD:C_0805_2012Metric, F.Cu at (122.4, 82.7)
- added C31: 100nF, Capacitor_SMD:C_0805_2012Metric, F.Cu at (122.5, 58.3)
- added C34: 100nF, Capacitor_SMD:C_0805_2012Metric, F.Cu at (123.8, 94.6)
- added C34: 100nF, Capacitor_SMD:C_0805_2012Metric, F.Cu at (123.8, 70.1)
- added C34: 100nF, Capacitor_SMD:C_0805_2012Metric, F.Cu at (123.9, 45.7)
- added C35: 100nF, Capacitor_SMD:C_0805_2012Metric, F.Cu at (115.5, 92.6)
- added C35: 100nF, Capacitor_SMD:C_0805_2012Metric, F.Cu at (115.5, 68.1)
- added C35: 100nF, Capacitor_SMD:C_0805_2012Metric, F.Cu at (115.5, 43.7)
- added C39: 100nF, Capacitor_SMD:C_0805_2012Metric, F.Cu at (54.1, 103.0)
- added C39: 100nF, Capacitor_SMD:C_0805_2012Metric, F.Cu at (55.3, 78.7)
- added C39: 100nF, Capacitor_SMD:C_0805_2012Metric, F.Cu at (55.8, 54.3)
- added C41: 100nF, Capacitor_SMD:C_1210_3225Metric, F.Cu at (55.9, 58.7)
- added C6: 4.7uF, Capacitor_SMD:C_1210_3225Metric, F.Cu at (92.0, 111.9)
- added C6: 4.7uF, Capacitor_SMD:C_1210_3225Metric, F.Cu at (91.9, 87.5)
- added C6: 4.7uF, Capacitor_SMD:C_1210_3225Metric, F.Cu at (92.0, 63.2)
- added C6: 4.7uF, Capacitor_SMD:C_1210_3225Metric, F.Cu at (85.8, 63.1)
- added C6: 4.7uF, Capacitor_SMD:C_1210_3225Metric, F.Cu at (85.7, 87.5)
- added C6: 4.7uF, Capacitor_SMD:C_1210_3225Metric, F.Cu at (85.9, 111.9)
- added C8: 4.7uF, Capacitor_SMD:C_1210_3225Metric, F.Cu at (95.1, 111.9)
- added C8: 4.7uF, Capacitor_SMD:C_1210_3225Metric, F.Cu at (95.0, 87.5)
- added C8: 4.7uF, Capacitor_SMD:C_1210_3225Metric, F.Cu at (95.1, 63.2)
- added C8: 4.7uF, Capacitor_SMD:C_1210_3225Metric, F.Cu at (88.9, 63.1)
- added C8: 4.7uF, Capacitor_SMD:C_1210_3225Metric, F.Cu at (88.8, 87.5)
- added C8: 4.7uF, Capacitor_SMD:C_1210_3225Metric, F.Cu at (89.0, 111.9)
- added Cs4: C_Small, Capacitor_SMD:C_0805_2012Metric, F.Cu at (80.8, 100.8)
- added Cs4: C_Small, Capacitor_SMD:C_0805_2012Metric, F.Cu at (80.8, 76.3)
- added Cs4: C_Small, Capacitor_SMD:C_0805_2012Metric, F.Cu at (80.9, 52.0)
- added D4: STPS0520Z, Diode_SMD:D_SOD-123, F.Cu at (63.4, 107.3)
- added D4: STPS0520Z, Diode_SMD:D_SOD-123, F.Cu at (63.4, 82.8)
- added D4: STPS0520Z, Diode_SMD:D_SOD-123, F.Cu at (63.5, 58.4)
- added D5: STPS0520Z, Diode_SMD:D_SOD-123, F.Cu at (70.1, 107.3)
- added D5: STPS0520Z, Diode_SMD:D_SOD-123, F.Cu at (70.1, 82.8)
- added D5: STPS0520Z, Diode_SMD:D_SOD-123, F.Cu at (70.2, 58.4)
- added D_L2: STTH1002CB, Diode_SMD:D_SOD-123, F.Cu at (78.4, 98.3)
- added D_L2: STTH1002CB, Diode_SMD:D_SOD-123, F.Cu at (78.4, 73.8)
- added D_L2: STTH1002CB, Diode_SMD:D_SOD-123, F.Cu at (78.5, 49.4)
- added J10: Conn_01x01, Footprints:0906_millmax, B.Cu at (126.2, 62.7)
- added J13: Conn_01x01, Footprints:0906_millmax, B.Cu at (126.2, 60.2)
- added J16: Conn_01x01, Footprints:0906_millmax, B.Cu at (126.5, 86.1)
- added J16: Conn_01x01, Footprints:0906_millmax, B.Cu at (122.2, 111.5)
- added J16: Conn_01x01, Footprints:0906_millmax, B.Cu at (132.7, 85.4)
- added J16: Conn_01x01, Footprints:0906_millmax, B.Cu at (132.7, 88.8)
- added J19: Conn_01x01, Footprints:0906_millmax, B.Cu at (126.5, 83.9)
- added J19: Conn_01x01, Footprints:0906_millmax, B.Cu at (122.2, 109.3)
- added J19: Conn_01x01, Footprints:0906_millmax, B.Cu at (130.5, 85.4)
- added J19: Conn_01x01, Footprints:0906_millmax, B.Cu at (130.5, 88.8)
- added J21: Conn_01x01, Footprints:0906_millmax, B.Cu at (65.2, 110.0)
- added J21: Conn_01x01, Footprints:0906_millmax, B.Cu at (65.2, 85.5)
- added J21: Conn_01x01, Footprints:0906_millmax, B.Cu at (65.3, 61.1)
- added J22: Conn_01x01, Footprints:0906_millmax, B.Cu at (62.4, 110.0)
- added J22: Conn_01x01, Footprints:0906_millmax, B.Cu at (62.4, 85.5)
- added J22: Conn_01x01, Footprints:0906_millmax, B.Cu at (62.5, 61.1)
- added J23: Conn_01x01, Footprints:0906_millmax, B.Cu at (71.7, 110.0)
- added J23: Conn_01x01, Footprints:0906_millmax, B.Cu at (71.7, 85.5)
- added J23: Conn_01x01, Footprints:0906_millmax, B.Cu at (71.8, 61.1)
- added J24: Conn_01x01, Footprints:0906_millmax, B.Cu at (68.8, 110.0)
- added J24: Conn_01x01, Footprints:0906_millmax, B.Cu at (68.8, 85.5)
- added J24: Conn_01x01, Footprints:0906_millmax, B.Cu at (68.9, 61.1)
- added J27: Conn_01x01, Footprints:0906_millmax, B.Cu at (126.5, 72.7)
- added J28: Conn_01x01, Footprints:0906_millmax, B.Cu at (126.1, 50.1)
- added J29: Conn_01x01, Footprints:0906_millmax, B.Cu at (126.1, 48.0)
- added J3: Conn_01x01, Footprints:0906_millmax, B.Cu at (108.8, 2.90)
- added J3: Conn_01x01, Footprints:0906_millmax, B.Cu at (107.3, 55.6)
- added J32: Conn_01x01, Footprints:0906_millmax, B.Cu at (126.5, 74.7)
- added J34: Conn_01x01, Footprints:0906_millmax, B.Cu at (106.2, 2.90)
- added J34: Conn_01x01, Footprints:0906_millmax, B.Cu at (104.7, 55.6)
- added L2: 33uH, Footprints:SRP1510CA-330M, F.Cu at (91.1, 99.5)
- added L2: 33uH, Footprints:SRP1510CA-330M, F.Cu at (91.1, 75.0)
- added L2: 33uH, Footprints:SRP1510CA-330M, F.Cu at (91.2, 50.6)
- added Q3: IPD200N15N3, Package_TO_SOT_SMD:TO-252-2, F.Cu at (78.0, 109.3)
- added Q3: IPD200N15N3, Package_TO_SOT_SMD:TO-252-2, F.Cu at (78.0, 84.4)
- added Q3: IPD200N15N3, Package_TO_SOT_SMD:TO-252-2, F.Cu at (78.1, 60.2)
- added Q4: IPD200N15N3, Package_TO_SOT_SMD:TO-252-2, F.Cu at (60.3, 98.9)
- added Q4: IPD200N15N3, Package_TO_SOT_SMD:TO-252-2, F.Cu at (60.3, 74.4)
- added Q4: IPD200N15N3, Package_TO_SOT_SMD:TO-252-2, F.Cu at (60.4, 50.0)
- added Q5: IPD200N15N3, Package_TO_SOT_SMD:TO-252-2, F.Cu at (73.5, 96.7)
- added Q5: IPD200N15N3, Package_TO_SOT_SMD:TO-252-2, F.Cu at (73.5, 72.2)
- added Q5: IPD200N15N3, Package_TO_SOT_SMD:TO-252-2, F.Cu at (73.6, 47.8)
- added R10: 27k, Resistor_SMD:R_0805_2012Metric, F.Cu at (119.6, 99.6)
- added R10: 27k, Resistor_SMD:R_0805_2012Metric, F.Cu at (119.6, 75.1)
- added R10: 27k, Resistor_SMD:R_0805_2012Metric, F.Cu at (119.7, 50.7)
- added R14: 12k, Resistor_SMD:R_0805_2012Metric, F.Cu at (120.5, 94.6)
- added R14: 12k, Resistor_SMD:R_0805_2012Metric, F.Cu at (120.5, 70.1)
- added R14: 12k, Resistor_SMD:R_0805_2012Metric, F.Cu at (120.6, 45.7)
- added R17: 12k, Resistor_SMD:R_0805_2012Metric, F.Cu at (122.9, 100.3)
- added R17: 12k, Resistor_SMD:R_0805_2012Metric, F.Cu at (122.9, 75.8)
- added R17: 12k, Resistor_SMD:R_0805_2012Metric, F.Cu at (123.0, 51.4)
- added R23: 200k, Resistor_SMD:R_0805_2012Metric, F.Cu at (115.4, 108.7)
- added R23: 200k, Resistor_SMD:R_0805_2012Metric, F.Cu at (117.7, 84.2)
- added R23: 200k, Resistor_SMD:R_0805_2012Metric, F.Cu at (117.8, 59.8)
- added R24: 200k, Resistor_SMD:R_0805_2012Metric, F.Cu at (115.4, 110.8)
- added R24: 200k, Resistor_SMD:R_0805_2012Metric, F.Cu at (117.7, 86.3)
- added R24: 200k, Resistor_SMD:R_0805_2012Metric, F.Cu at (117.8, 61.9)
- added R26: 82k, Resistor_SMD:R_0805_2012Metric, F.Cu at (118.2, 107.2)
- added R26: 82k, Resistor_SMD:R_0805_2012Metric, F.Cu at (120.5, 82.7)
- added R26: 82k, Resistor_SMD:R_0805_2012Metric, F.Cu at (120.6, 58.3)
- added R28: 82k, Resistor_SMD:R_0805_2012Metric, F.Cu at (119.1, 112.8)
- added R28: 82k, Resistor_SMD:R_0805_2012Metric, F.Cu at (121.4, 88.3)
- added R28: 82k, Resistor_SMD:R_0805_2012Metric, F.Cu at (121.5, 63.9)
- added R33: 0, Resistor_SMD:R_0805_2012Metric, F.Cu at (62.3, 104.4)
- added R33: 0, Resistor_SMD:R_0805_2012Metric, F.Cu at (62.3, 79.9)
- added R33: 0, Resistor_SMD:R_0805_2012Metric, F.Cu at (62.4, 55.5)
- added R34: 0, Resistor_SMD:R_0805_2012Metric, F.Cu at (69.0, 104.4)
- added R34: 0, Resistor_SMD:R_0805_2012Metric, F.Cu at (69.0, 79.9)
- added R34: 0, Resistor_SMD:R_0805_2012Metric, F.Cu at (69.1, 55.5)
- added R35: 1k, Resistor_SMD:R_0805_2012Metric, F.Cu at (67.2, 100.3)
- added R35: 1k, Resistor_SMD:R_0805_2012Metric, F.Cu at (67.2, 75.8)
- added R35: 1k, Resistor_SMD:R_0805_2012Metric, F.Cu at (67.3, 51.4)
- added R36: 1k, Resistor_SMD:R_0805_2012Metric, F.Cu at (73.1, 102.5)
- added R36: 1k, Resistor_SMD:R_0805_2012Metric, F.Cu at (73.1, 78.0)
- added R36: 1k, Resistor_SMD:R_0805_2012Metric, F.Cu at (73.2, 53.6)
- added R5: 2,2, Resistor_SMD:R_0805_2012Metric, F.Cu at (64.2, 104.4)
- added R5: 2,2, Resistor_SMD:R_0805_2012Metric, F.Cu at (64.2, 79.9)
- added R5: 2,2, Resistor_SMD:R_0805_2012Metric, F.Cu at (64.3, 55.5)
- added R6: 2,2, Resistor_SMD:R_0805_2012Metric, F.Cu at (71.2, 104.4)
- added R6: 2,2, Resistor_SMD:R_0805_2012Metric, F.Cu at (71.2, 79.9)
- added R6: 2,2, Resistor_SMD:R_0805_2012Metric, F.Cu at (71.3, 55.5)
- added R9: 27k, Resistor_SMD:R_0805_2012Metric, F.Cu at (119.6, 97.3)
- added R9: 27k, Resistor_SMD:R_0805_2012Metric, F.Cu at (119.6, 72.8)
- added R9: 27k, Resistor_SMD:R_0805_2012Metric, F.Cu at (119.7, 48.4)
- added REF**: C_1812_4532Metric, Capacitor_SMD:C_1812_4532Metric, F.Cu at (56.5, 81.8)
- added REF**: C_1812_4532Metric, Capacitor_SMD:C_1812_4532Metric, F.Cu at (55.5, 106.2)
- added Rs4: R_Small, Resistor_SMD:R_0805_2012Metric, F.Cu at (80.8, 97.6)
- added Rs4: R_Small, Resistor_SMD:R_0805_2012Metric, F.Cu at (80.8, 73.1)
- added Rs4: R_Small, Resistor_SMD:R_0805_2012Metric, F.Cu at (80.9, 48.7)
- added Rv3: 150K, Resistor_SMD:R_0805_2012Metric, F.Cu at (104.6, 95.3)
- added Rv3: 150K, Resistor_SMD:R_0805_2012Metric, F.Cu at (104.6, 70.8)
- added Rv3: 150K, Resistor_SMD:R_0805_2012Metric, F.Cu at (104.7, 46.4)
- added Rv4: 470, Resistor_SMD:R_0805_2012Metric, F.Cu at (104.6, 98.5)
- added Rv4: 470, Resistor_SMD:R_0805_2012Metric, F.Cu at (104.6, 74.0)
- added Rv4: 470, Resistor_SMD:R_0805_2012Metric, F.Cu at (104.7, 49.6)
- added U11: OPA316, Package_TO_SOT_SMD:SOT-353_SC-70-5, F.Cu at (119.2, 110.3)
- added U11: OPA316, Package_TO_SOT_SMD:SOT-353_SC-70-5, F.Cu at (121.5, 85.8)
- added U11: OPA316, Package_TO_SOT_SMD:SOT-353_SC-70-5, F.Cu at (121.6, 61.4)
- added U4: ACS730xLCTR-20AB, Package_SO:SOIC-8_3.9x4.9mm_P1.27mm, F.Cu at (106.7, 108.7)
- added U4: ACS730xLCTR-20AB, Package_SO:SOIC-8_3.9x4.9mm_P1.27mm, F.Cu at (106.8, 84.7)
- added U4: ACS730xLCTR-20AB, Package_SO:SOIC-8_3.9x4.9mm_P1.27mm, F.Cu at (106.9, 60.3)
- added U6: AMC1100DUB, Footprints:SOP-8_6.62x9.15mm_P2.54mm, F.Cu at (111.7, 98.5)
- added U6: AMC1100DUB, Footprints:SOP-8_6.62x9.15mm_P2.54mm, F.Cu at (111.7, 74.0)
- added U6: AMC1100DUB, Footprints:SOP-8_6.62x9.15mm_P2.54mm, F.Cu at (111.8, 49.6)
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Routing:
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- added copper zone on F.Cu, net (none)
- added copper zone on In1.Cu, net (none)
- added copper zone on In2.Cu, net (none)
- added copper zone on B.Cu, net /N
- added copper zone on B.Cu, net /SW_Node2
- added copper zone on B.Cu, net /V_Out
- added copper zone on F.Cu, net Net-(C13-Pad2)
Other:
- net class Default removed
